File: kicad/keyboard.sch (KiCad schematic (older format))
At the start: 159 parts, among them J1 USB_mini_micro_B, U1 ATMEGA32U4

Commit message: Updated project
Parts:
- removed C8: 1u, Capacitor_SMD:C_0805_2012Metric_Pad1.15x1.40mm_HandSolder, symbol Device:C_Small
- removed D_1, D_2, D_A, D_B, D_BACKSPACE, D_C, D_COMMA, D_D, D_DOWN, D_E, D_ESC, D_F, D_F10, D_F11, D_F12, D_G, D_H, D_LEFT, D_M, D_N, D_Q, D_QUOTE, D_R, D_RIGHT, D_S, D_TAB, D_V, D_W: D, keyboard_parts:D_SOD123_axial, symbol Device:D
- removed J1: USB_mini_micro_B, keyboard_parts:USB_miniB_hirose_5S8, symbol keyboard_parts:USB_mini_micro_B
- removed K_1, K_2, K_A, K_B, K_C, K_COMMA, K_D, K_DOWN, K_E, K_F, K_F10, K_F11, K_F12, K_G, K_H, K_LEFT, K_M, K_N, K_Q, K_QUOTE, K_R, K_RIGHT, K_S, K_V, K_W: KEYSW, MX_Alps_Hybrid:MX-1U-NoLED, symbol keyboard_parts:KEYSW
- removed K_BACKSPACE: KEYSW, MX_Alps_Hybrid:MX-2U-NoLED, symbol keyboard_parts:KEYSW
- removed K_TAB: KEYSW, MX_Alps_Hybrid:MX-1.5U-NoLED, symbol keyboard_parts:KEYSW
- removed R3 (x2): 22, Resistor_SMD:R_0805_2012Metric_Pad1.15x1.40mm_HandSolder, symbol Device:R
- removed U1: ATMEGA32U4, Package_QFP:TQFP-44_10x10mm_P0.8mm, symbol keyboard_parts:ATMEGA32U4
- added D_0, D_50, D_51, D_52, D_53, D_54, D_55, D_56, D_57, D_58, D_59, D_60, D_61, D_62, D_63, D_64, D_65, D_66, D_67, D_68, D_69, D_70, D_71, D_72, D_73, D_74, D_75, D_76: D, Diode_SMD:D_SOD-123, symbol Device:D_Small
- added K_50, K_51, K_52, K_53, K_55, K_56, K_57, K_58, K_59, K_60, K_61, K_62, K_63, K_64, K_65, K_66, K_67, K_73, K_74, K_75, K_76: KEYSW, MX_Alps_Hybrid:MX-1U-NoLED, symbol MX_Alps_Hybrid:MX-NoLED
- added K_54, K_68, K_69, K_70, K_72: KEYSW, MX_Alps_Hybrid:MX-1.25U-NoLED, symbol MX_Alps_Hybrid:MX-NoLED
- added K_71: KEYSW, MX_Alps_Hybrid:MX-6.25U-NoLED, symbol MX_Alps_Hybrid:MX-NoLED
- D_1: renamed from D_F1; footprint keyboard_parts:D_SOD123_axial -> Diode_SMD:D_SOD-123; symbol Device:D -> Device:D_Small
- D_10: renamed from D_3; footprint keyboard_parts:D_SOD123_axial -> Diode_SMD:D_SOD-123; symbol Device:D -> Device:D_Small
- D_11: renamed from D_4; footprint keyboard_parts:D_SOD123_axial -> Diode_SMD:D_SOD-123; symbol Device:D -> Device:D_Small
- D_12: renamed from D_5; footprint keyboard_parts:D_SOD123_axial -> Diode_SMD:D_SOD-123; symbol Device:D -> Device:D_Small
- D_13: renamed from D_6; footprint keyboard_parts:D_SOD123_axial -> Diode_SMD:D_SOD-123; symbol Device:D -> Device:D_Small
- D_14: renamed from D_7; footprint keyboard_parts:D_SOD123_axial -> Diode_SMD:D_SOD-123; symbol Device:D -> Device:D_Small
- D_15: renamed from D_8; footprint keyboard_parts:D_SOD123_axial -> Diode_SMD:D_SOD-123; symbol Device:D -> Device:D_Small
- D_16: renamed from D_9; footprint keyboard_parts:D_SOD123_axial -> Diode_SMD:D_SOD-123; symbol Device:D -> Device:D_Small
- D_17: renamed from D_0; footprint keyboard_parts:D_SOD123_axial -> Diode_SMD:D_SOD-123; symbol Device:D -> Device:D_Small
- D_18: renamed from D_MINUS; footprint keyboard_parts:D_SOD123_axial -> Diode_SMD:D_SOD-123; symbol Device:D -> Device:D_Small
- D_19: renamed from D_EQUAL; footprint keyboard_parts:D_SOD123_axial -> Diode_SMD:D_SOD-123; symbol Device:D -> Device:D_Small
- D_2: renamed from D_F2; footprint keyboard_parts:D_SOD123_axial -> Diode_SMD:D_SOD-123; symbol Device:D -> Device:D_Small
- D_20: renamed from D_T; footprint keyboard_parts:D_SOD123_axial -> Diode_SMD:D_SOD-123; symbol Device:D -> Device:D_Small
- D_21: renamed from D_Y; footprint keyboard_parts:D_SOD123_axial -> Diode_SMD:D_SOD-123; symbol Device:D -> Device:D_Small
- D_22: renamed from D_U; footprint keyboard_parts:D_SOD123_axial -> Diode_SMD:D_SOD-123; symbol Device:D -> Device:D_Small
- D_23: renamed from D_I; footprint keyboard_parts:D_SOD123_axial -> Diode_SMD:D_SOD-123; symbol Device:D -> Device:D_Small
- D_24: renamed from D_O; footprint keyboard_parts:D_SOD123_axial -> Diode_SMD:D_SOD-123; symbol Device:D -> Device:D_Small
- D_25: renamed from D_P; footprint keyboard_parts:D_SOD123_axial -> Diode_SMD:D_SOD-123; symbol Device:D -> Device:D_Small
- D_26: renamed from D_ACC; footprint keyboard_parts:D_SOD123_axial -> Diode_SMD:D_SOD-123; symbol Device:D -> Device:D_Small
- D_27: renamed from D_CBRAC; footprint keyboard_parts:D_SOD123_axial -> Diode_SMD:D_SOD-123; symbol Device:D -> Device:D_Small
- D_28: renamed from D_ENTER; footprint keyboard_parts:D_SOD123_axial -> Diode_SMD:D_SOD-123; symbol Device:D -> Device:D_Small
- D_29: renamed from D_CAPS; footprint keyboard_parts:D_SOD123_axial -> Diode_SMD:D_SOD-123; symbol Device:D -> Device:D_Small
- D_3: renamed from D_F3; footprint keyboard_parts:D_SOD123_axial -> Diode_SMD:D_SOD-123; symbol Device:D -> Device:D_Small
- D_30: renamed from D_J; footprint keyboard_parts:D_SOD123_axial -> Diode_SMD:D_SOD-123; symbol Device:D -> Device:D_Small
- D_31: renamed from D_K; footprint keyboard_parts:D_SOD123_axial -> Diode_SMD:D_SOD-123; symbol Device:D -> Device:D_Small
- D_32: renamed from D_L; footprint keyboard_parts:D_SOD123_axial -> Diode_SMD:D_SOD-123; symbol Device:D -> Device:D_Small
- D_33: renamed from D_Ç; footprint keyboard_parts:D_SOD123_axial -> Diode_SMD:D_SOD-123; symbol Device:D -> Device:D_Small
- D_34: renamed from D_TILDE; footprint keyboard_parts:D_SOD123_axial -> Diode_SMD:D_SOD-123; symbol Device:D -> Device:D_Small
- D_35: renamed from D_OBRAC; footprint keyboard_parts:D_SOD123_axial -> Diode_SMD:D_SOD-123; symbol Device:D -> Device:D_Small
- D_36: renamed from D_SHIFT; footprint keyboard_parts:D_SOD123_axial -> Diode_SMD:D_SOD-123; symbol Device:D -> Device:D_Small
- D_37: renamed from D_BSLSH; footprint keyboard_parts:D_SOD123_axial -> Diode_SMD:D_SOD-123; symbol Device:D -> Device:D_Small
- D_38: renamed from D_Z; footprint keyboard_parts:D_SOD123_axial -> Diode_SMD:D_SOD-123; symbol Device:D -> Device:D_Small
- D_39: renamed from D_X; footprint keyboard_parts:D_SOD123_axial -> Diode_SMD:D_SOD-123; symbol Device:D -> Device:D_Small
- D_4: renamed from D_F4; footprint keyboard_parts:D_SOD123_axial -> Diode_SMD:D_SOD-123; symbol Device:D -> Device:D_Small
- D_40: renamed from D_DOT; footprint keyboard_parts:D_SOD123_axial -> Diode_SMD:D_SOD-123; symbol Device:D -> Device:D_Small
- D_41: renamed from D_SEMIC; footprint keyboard_parts:D_SOD123_axial -> Diode_SMD:D_SOD-123; symbol Device:D -> Device:D_Small
- D_42: renamed from D_SLASH; footprint keyboard_parts:D_SOD123_axial -> Diode_SMD:D_SOD-123; symbol Device:D -> Device:D_Small
- D_43: renamed from D_UP; footprint keyboard_parts:D_SOD123_axial -> Diode_SMD:D_SOD-123; symbol Device:D -> Device:D_Small
- D_44: renamed from D_CTRL; footprint keyboard_parts:D_SOD123_axial -> Diode_SMD:D_SOD-123; symbol Device:D -> Device:D_Small
- D_45: renamed from D_GUI; footprint keyboard_parts:D_SOD123_axial -> Diode_SMD:D_SOD-123; symbol Device:D -> Device:D_Small
- D_46: renamed from D_ALT; footprint keyboard_parts:D_SOD123_axial -> Diode_SMD:D_SOD-123; symbol Device:D -> Device:D_Small
- D_47: renamed from D_SPACE; footprint keyboard_parts:D_SOD123_axial -> Diode_SMD:D_SOD-123; symbol Device:D -> Device:D_Small
- D_48: renamed from D_APP; footprint keyboard_parts:D_SOD123_axial -> Diode_SMD:D_SOD-123; symbol Device:D -> Device:D_Small
- D_49: renamed from D_DEL; footprint keyboard_parts:D_SOD123_axial -> Diode_SMD:D_SOD-123; symbol Device:D -> Device:D_Small
- D_5: renamed from D_F5; footprint keyboard_parts:D_SOD123_axial -> Diode_SMD:D_SOD-123; symbol Device:D -> Device:D_Small
- D_6: renamed from D_F6; footprint keyboard_parts:D_SOD123_axial -> Diode_SMD:D_SOD-123; symbol Device:D -> Device:D_Small
- D_7: renamed from D_F7; footprint keyboard_parts:D_SOD123_axial -> Diode_SMD:D_SOD-123; symbol Device:D -> Device:D_Small
- D_8: renamed from D_F8; footprint keyboard_parts:D_SOD123_axial -> Diode_SMD:D_SOD-123; symbol Device:D -> Device:D_Small
- D_9: renamed from D_F9; footprint keyboard_parts:D_SOD123_axial -> Diode_SMD:D_SOD-123; symbol Device:D -> Device:D_Small
- K_0: renamed from K_ESC; symbol keyboard_parts:KEYSW -> MX_Alps_Hybrid:MX-NoLED
- K_1: renamed from K_F1; symbol keyboard_parts:KEYSW -> MX_Alps_Hybrid:MX-NoLED
- K_10: renamed from K_3; symbol keyboard_parts:KEYSW -> MX_Alps_Hybrid:MX-NoLED
- K_11: renamed from K_4; symbol keyboard_parts:KEYSW -> MX_Alps_Hybrid:MX-NoLED
- K_12: renamed from K_5; symbol keyboard_parts:KEYSW -> MX_Alps_Hybrid:MX-NoLED
- K_13: renamed from K_6; symbol keyboard_parts:KEYSW -> MX_Alps_Hybrid:MX-NoLED
- K_14: renamed from K_7; symbol keyboard_parts:KEYSW -> MX_Alps_Hybrid:MX-NoLED
- K_15: renamed from K_8; symbol keyboard_parts:KEYSW -> MX_Alps_Hybrid:MX-NoLED
- K_16: renamed from K_9; symbol keyboard_parts:KEYSW -> MX_Alps_Hybrid:MX-NoLED
- K_17: renamed from K_0; symbol keyboard_parts:KEYSW -> MX_Alps_Hybrid:MX-NoLED
- K_18: renamed from K_MINUS; symbol keyboard_parts:KEYSW -> MX_Alps_Hybrid:MX-NoLED
- K_19: renamed from K_EQUAL; symbol keyboard_parts:KEYSW -> MX_Alps_Hybrid:MX-NoLED
- K_2: renamed from K_F2; symbol keyboard_parts:KEYSW -> MX_Alps_Hybrid:MX-NoLED
- K_20: renamed from K_T; symbol keyboard_parts:KEYSW -> MX_Alps_Hybrid:MX-NoLED
- K_21: renamed from K_Y; symbol keyboard_parts:KEYSW -> MX_Alps_Hybrid:MX-NoLED
- K_22: renamed from K_U; symbol keyboard_parts:KEYSW -> MX_Alps_Hybrid:MX-NoLED
- K_23: renamed from K_I; symbol keyboard_parts:KEYSW -> MX_Alps_Hybrid:MX-NoLED
- K_24: renamed from K_O; symbol keyboard_parts:KEYSW -> MX_Alps_Hybrid:MX-NoLED
- K_25: renamed from K_P; symbol keyboard_parts:KEYSW -> MX_Alps_Hybrid:MX-NoLED
- K_26: renamed from K_ACC; footprint MX_Alps_Hybrid:MX-1U-NoLED -> MX_Alps_Hybrid:MX-2U-NoLED; symbol keyboard_parts:KEYSW -> MX_Alps_Hybrid:MX-NoLED
- K_27: renamed from K_CBRAC; footprint MX_Alps_Hybrid:MX-1U-NoLED -> MX_Alps_Hybrid:MX-1.5U-NoLED; symbol keyboard_parts:KEYSW -> MX_Alps_Hybrid:MX-NoLED
- K_28: renamed from K_ENTER; footprint MX_Alps_Hybrid:MX-1.25U-NoLED -> MX_Alps_Hybrid:MX-1U-NoLED; symbol keyboard_parts:KEYSW -> MX_Alps_Hybrid:MX-NoLED
- K_29: renamed from K_CAPS; footprint MX_Alps_Hybrid:MX-1.75U-NoLED -> MX_Alps_Hybrid:MX-1U-NoLED; symbol keyboard_parts:KEYSW -> MX_Alps_Hybrid:MX-NoLED
- K_3: renamed from K_F3; symbol keyboard_parts:KEYSW -> MX_Alps_Hybrid:MX-NoLED
- K_30: renamed from K_J; symbol keyboard_parts:KEYSW -> MX_Alps_Hybrid:MX-NoLED
- K_31: renamed from K_K; symbol keyboard_parts:KEYSW -> MX_Alps_Hybrid:MX-NoLED
- K_32: renamed from K_L; symbol keyboard_parts:KEYSW -> MX_Alps_Hybrid:MX-NoLED
- K_33: renamed from K_Ç; symbol keyboard_parts:KEYSW -> MX_Alps_Hybrid:MX-NoLED
- K_34: renamed from K_TILDE; symbol keyboard_parts:KEYSW -> MX_Alps_Hybrid:MX-NoLED
- K_35: renamed from K_OBRAC; symbol keyboard_parts:KEYSW -> MX_Alps_Hybrid:MX-NoLED
- K_36: renamed from K_SHIFT; footprint MX_Alps_Hybrid:MX-1.25U-NoLED -> MX_Alps_Hybrid:MX-1U-NoLED; symbol keyboard_parts:KEYSW -> MX_Alps_Hybrid:MX-NoLED
- K_37: renamed from K_BSLSH; symbol keyboard_parts:KEYSW -> MX_Alps_Hybrid:MX-NoLED
- K_38: renamed from K_Z; symbol keyboard_parts:KEYSW -> MX_Alps_Hybrid:MX-NoLED
- K_39: renamed from K_X; symbol keyboard_parts:KEYSW -> MX_Alps_Hybrid:MX-NoLED
- K_4: renamed from K_F4; symbol keyboard_parts:KEYSW -> MX_Alps_Hybrid:MX-NoLED
- K_40: renamed from K_DOT; footprint MX_Alps_Hybrid:MX-1U-NoLED -> MX_Alps_Hybrid:MX-1.25U-NoLED; symbol keyboard_parts:KEYSW -> MX_Alps_Hybrid:MX-NoLED
- K_41: renamed from K_SEMIC; footprint MX_Alps_Hybrid:MX-1U-NoLED -> MX_Alps_Hybrid:MX-1.75U-NoLED; symbol keyboard_parts:KEYSW -> MX_Alps_Hybrid:MX-NoLED
- K_42: renamed from K_SLASH; symbol keyboard_parts:KEYSW -> MX_Alps_Hybrid:MX-NoLED
- K_43: renamed from K_UP; symbol keyboard_parts:KEYSW -> MX_Alps_Hybrid:MX-NoLED
- K_44: renamed from K_CTRL; footprint MX_Alps_Hybrid:MX-1.25U-NoLED -> MX_Alps_Hybrid:MX-1U-NoLED; symbol keyboard_parts:KEYSW -> MX_Alps_Hybrid:MX-NoLED
- K_45: renamed from K_GUI; footprint MX_Alps_Hybrid:MX-1.25U-NoLED -> MX_Alps_Hybrid:MX-1U-NoLED; symbol keyboard_parts:KEYSW -> MX_Alps_Hybrid:MX-NoLED
- K_46: renamed from K_ALT; footprint MX_Alps_Hybrid:MX-1.25U-NoLED -> MX_Alps_Hybrid:MX-1U-NoLED; symbol keyboard_parts:KEYSW -> MX_Alps_Hybrid:MX-NoLED
- K_47: renamed from K_SPACE; footprint MX_Alps_Hybrid:MX-6.25U-NoLED -> MX_Alps_Hybrid:MX-1U-NoLED; symbol keyboard_parts:KEYSW -> MX_Alps_Hybrid:MX-NoLED
- K_48: renamed from K_APP; footprint MX_Alps_Hybrid:MX-1.25U-NoLED -> MX_Alps_Hybrid:MX-1U-NoLED; symbol keyboard_parts:KEYSW -> MX_Alps_Hybrid:MX-NoLED
- K_49: renamed from K_DEL; symbol keyboard_parts:KEYSW -> MX_Alps_Hybrid:MX-NoLED
- K_5: renamed from K_F5; symbol keyboard_parts:KEYSW -> MX_Alps_Hybrid:MX-NoLED
- K_6: renamed from K_F6; symbol keyboard_parts:KEYSW -> MX_Alps_Hybrid:MX-NoLED
- K_7: renamed from K_F7; symbol keyboard_parts:KEYSW -> MX_Alps_Hybrid:MX-NoLED
- K_8: renamed from K_F8; symbol keyboard_parts:KEYSW -> MX_Alps_Hybrid:MX-NoLED
- K_9: renamed from K_F9; symbol keyboard_parts:KEYSW -> MX_Alps_Hybrid:MX-NoLED
Connections:
- net col0: now also K_13.1 (COL), K_27.1 (COL), K_41.1 (COL), K_54.1 (COL), K_68.1 (COL); no longer K_29.1, K_36.1, K_44.1
- net col1: now also K_14.1 (COL), K_28.1 (COL), K_42.1 (COL), K_55.1 (COL), K_69.1 (COL); no longer K_37.1, K_45.1
- net col10: now also K_23.1 (COL), K_37.1 (COL), K_51.1 (COL), K_64.1 (COL), K_73.1 (COL); no longer K_17.1, K_25.1, K_33.1, K_40.1, K_49.1
- net col11: now also K_10.1 (COL), K_24.1 (COL), K_38.1 (COL), K_52.1 (COL), K_65.1 (COL), K_74.1 (COL); no longer K_18.1, K_26.1, K_34.1, K_41.1
- net col12: now also K_11.1 (COL), K_25.1 (COL), K_39.1 (COL), K_53.1 (COL), K_66.1 (COL), K_75.1 (COL); no longer K_19.1, K_27.1, K_35.1, K_42.1
- net col13: now also K_12.1 (COL), K_26.1 (COL), K_40.1 (COL), K_67.1 (COL), K_76.1 (COL); no longer K_28.1, K_43.1
- net col2: now also K_15.1 (COL), K_29.1 (COL), K_43.1 (COL), K_56.1 (COL), K_70.1 (COL); no longer K_38.1, K_46.1
- net col3: now also K_16.1 (COL), K_30.1 (COL), K_44.1 (COL), K_57.1 (COL); no longer K_10.1, K_39.1
- net col4: now also K_17.1 (COL), K_31.1 (COL), K_45.1 (COL), K_58.1 (COL); no longer K_11.1
- net col5: now also K_18.1 (COL), K_32.1 (COL), K_46.1 (COL), K_59.1 (COL); no longer K_12.1, K_20.1
- net col6: now also K_19.1 (COL), K_33.1 (COL), K_60.1 (COL), K_71.1 (COL); no longer K_13.1, K_21.1
- net col7: now also K_20.1 (COL), K_34.1 (COL), K_48.1 (COL), K_61.1 (COL); no longer K_14.1, K_22.1, K_30.1
- net col8: now also K_21.1 (COL), K_35.1 (COL), K_49.1 (COL), K_62.1 (COL); no longer K_15.1, K_23.1, K_31.1
- net col9: now also K_22.1 (COL), K_36.1 (COL), K_50.1 (COL), K_63.1 (COL), K_72.1 (COL); no longer K_16.1, K_24.1, K_32.1, K_48.1
- net row0: now also D_10.1 (K), D_11.1 (K), D_12.1 (K), D_0.1 (K)
- net row1: now also D_20.1 (K), D_21.1 (K), D_22.1 (K), D_23.1 (K), D_24.1 (K), D_25.1 (K), D_26.1 (K); no longer D_10.1 (K), D_11.1 (K), D_12.1 (K)
- net row2: now also D_28.1 (K), D_29.1 (K), D_30.1 (K), D_31.1 (K), D_32.1 (K), D_33.1 (K), D_34.1 (K), D_35.1 (K), D_36.1 (K), D_37.1 (K), D_38.1 (K), D_39.1 (K), D_40.1 (K); no longer D_20.1 (K), D_21.1 (K), D_22.1 (K), D_23.1 (K), D_24.1 (K), D_25.1 (K), D_26.1 (K)
- net row3: now also D_41.1 (K), D_42.1 (K), D_43.1 (K), D_44.1 (K), D_45.1 (K), D_46.1 (K), D_47.1 (K), D_48.1 (K), D_49.1 (K), D_50.1 (K), D_51.1 (K), D_52.1 (K), D_53.1 (K); no longer D_28.1 (K), D_29.1 (K), D_30.1 (K), D_31.1 (K), D_32.1 (K), D_33.1 (K), D_34.1 (K), D_35.1 (K)
- net row4: now also D_54.1 (K), D_55.1 (K), D_56.1 (K), D_57.1 (K), D_58.1 (K), D_59.1 (K), D_60.1 (K), D_61.1 (K), D_62.1 (K), D_63.1 (K), D_64.1 (K), D_65.1 (K), D_66.1 (K), D_67.1 (K); no longer D_36.1 (K), D_37.1 (K), D_38.1 (K), D_39.1 (K), D_40.1 (K), D_41.1 (K), D_42.1 (K), D_43.1 (K)
- net row5: now also D_68.1 (K), D_69.1 (K), D_70.1 (K), D_71.1 (K), D_72.1 (K), D_73.1 (K), D_74.1 (K), D_75.1 (K), D_76.1 (K); no longer D_44.1 (K), D_45.1 (K), D_46.1 (K), D_47.1 (K), D_48.1 (K), D_49.1 (K)
- net at K_0.2 (ROW): now also D_0.2 (A)
- new net: D_50.2 (A), K_50.2 (ROW)
- new net: D_51.2 (A), K_51.2 (ROW)
- new net: D_52.2 (A), K_52.2 (ROW)
- new net: D_53.2 (A), K_53.2 (ROW)
- new net: D_54.2 (A), K_54.2 (ROW)
- new net: D_55.2 (A), K_55.2 (ROW)
- new net: D_56.2 (A), K_56.2 (ROW)
- new net: D_57.2 (A), K_57.2 (ROW)
- new net: D_58.2 (A), K_58.2 (ROW)
- new net: D_59.2 (A), K_59.2 (ROW)
- new net: D_60.2 (A), K_60.2 (ROW)
- new net: D_61.2 (A), K_61.2 (ROW)
- new net: D_62.2 (A), K_62.2 (ROW)
- new net: D_63.2 (A), K_63.2 (ROW)
- new net: D_64.2 (A), K_64.2 (ROW)
- new net: D_65.2 (A), K_65.2 (ROW)
- new net: D_66.2 (A), K_66.2 (ROW)
- new net: D_67.2 (A), K_67.2 (ROW)
- new net: D_68.2 (A), K_68.2 (ROW)
- new net: D_69.2 (A), K_69.2 (ROW)
- new net: D_70.2 (A), K_70.2 (ROW)
- new net: D_71.2 (A), K_71.2 (ROW)
- new net: D_72.2 (A), K_72.2 (ROW)
- new net: D_73.2 (A), K_73.2 (ROW)
- new net: D_74.2 (A), K_74.2 (ROW)
- new net: D_75.2 (A), K_75.2 (ROW)
- new net: D_76.2 (A), K_76.2 (ROW)
- no-connect marks 1 -> 0

Commit message: Schematic complete
Parts:
- added C1, C2: 22pF, Capacitor_SMD:C_0805_2012Metric, symbol Device:C_Small
- added C3: 1uF, Capacitor_SMD:C_0805_2012Metric, symbol Device:C_Small
- added C4, C5, C6: 0.1uF, Capacitor_SMD:C_0805_2012Metric, symbol Device:C_Small
- added C7: 10uF, Capacitor_SMD:C_0805_2012Metric, symbol Device:C_Small
- added F1: 500mA, Fuse:Fuse_1206_3216Metric, symbol Device:Polyfuse_Small
- added R1, R4: 10k, Resistor_SMD:R_0805_2012Metric, symbol Device:R_Small
- added R2, R3: 22, Resistor_SMD:R_0805_2012Metric, symbol Device:R_Small
- added SW1: SW_Push, random-keyboard-parts:SKQG-1155865, symbol Switch:SW_Push
- added U1: ATmega32U4-AU, Package_QFP:TQFP-44_10x10mm_P0.8mm, symbol MCU_Microchip_ATmega:ATmega32U4-AU
- added USB1: Molex-0548190589, random-keyboard-parts:Molex-0548190589, symbol random-keyboard-parts:Molex-0548190589
- added Y1: 16MHz, Crystal:Crystal_SMD_3225-4Pin_3.2x2.5mm, symbol Device:Crystal_GND24_Small
Connections:
- net col0: now also U1.30 (PB6)
- net col1: now also U1.12 (PB7)
- net col10: now also U1.26 (PD6)
- net col11: now also U1.27 (PD7)
- net col12: now also U1.1 (PE6)
- net col13: now also U1.41 (PF0)
- net col2: now also U1.31 (PC6)
- net col3: now also U1.32 (PC7)
- net col4: now also U1.18 (PD0)
- net col5: now also U1.19 (PD1)
- net col6: now also U1.20 (PD2)
- net col7: now also U1.21 (PD3)
- net col8: now also U1.25 (PD4)
- net col9: now also U1.22 (PD5)
- net row0: now also U1.8 (PB0)
- net row1: now also U1.9 (PB1)
- net row2: now also U1.10 (PB2)
- net row3: now also U1.11 (PB3)
- net row4: now also U1.28 (PB4)
- net row5: now also U1.29 (PB5)
- new net: R1.2, SW1.2, U1.13 (~RESET)
- new net: C2.1, U1.16 (XTAL2), Y1.3
- new net: C1.1, U1.17 (XTAL1), Y1.1
- new net: R3.1, U1.3 (D-)
- new net: R4.2, U1.33 (~HWB~/PE2)
- new net: R2.1, U1.4 (D+)
- new net: C3.1, U1.6 (UCAP)
- new net +5V: C4.1, C5.1, C6.1, C7.1, F1.1, R1.1, U1.14 (VCC), U1.2 (UVCC), U1.24 (AVCC), U1.34 (VCC), U1.44 (AVCC), U1.7 (VBUS)
- new net D+: R2.2, USB1.3 (D+)
- new net D-: R3.2, USB1.4 (D-)
- new net GND: C1.2, C2.2, C3.2, C4.2, C5.2, C6.2, C7.2, R4.1, SW1.1, U1.15 (GND), U1.23 (GND), U1.35 (GND), U1.43 (GND), U1.5 (UGND), USB1.1 (GND), Y1.2, Y1.4
- new net VCC: F1.2, USB1.5 (VBUS)

Commit message: 1st version of PCB complete
Parts:
- K_40: footprint MX_Alps_Hybrid:MX-1.25U-NoLED -> MX_Alps_Hybrid:MX-ISOEnter-NoLED
Changed lines of the file:
@@
 F 0 "K_40" H 14400 3233 60  0000 C CNN
 F 1 "KEYSW" H 14400 2900 60  0001 C CNN
-F 2 "MX_Alps_Hybrid:MX-1.25U-NoLED" H 14400 3000 60  0001 C CNN
+F 2 "MX_Alps_Hybrid:MX-ISOEnter-NoLED" H 14400 3000 60  0001 C CNN
 F 3 "" H 14400 3000 60  0000 C CNN
 	1    14400 3000
@@
 Wire Wire Line
 	2400 11750 2400 11900
-Text GLabel 1500 13300 0    50   Input ~ 0
+Text GLabel 1500 13300 0    50   Output ~ 0
 D+
-Text GLabel 1500 13400 0    50   Input ~ 0
+Text GLabel 1500 13400 0    50   Output ~ 0
 D-
 $Comp
