File: kicad/keyboard.kicad_pcb (KiCad board)
At the start: 2 copper layers, 295.5 x 124 mm, 174 parts, among them J1 USB_C_Receptacle_USB2.0, SW1 SW_Push, SW10 SW_Push, SW11 SW_Push, SW12 SW_Push, SW13 SW_Push, SW14 SW_Push, SW15 SW_Push, SW16 SW_Push, SW17 SW_Push, SW18 SW_Push, SW19 SW_Push, SW2 SW_Push, SW20 SW_Push, SW21 SW_Push, SW22 SW_Push, SW23 SW_Push, SW24 SW_Push, SW25 SW_Push, SW26 SW_Push, SW27 SW_Push, SW28 SW_Push, SW29 SW_Push, SW3 SW_Push, SW30 SW_Push, SW31 SW_Push, SW32 SW_Push, SW33 SW_Push, SW34 SW_Push, SW35 SW_Push, SW36 SW_Push, SW37 SW_Push, SW38 SW_Push, SW39 SW_Push, SW4 SW_Push, SW40 SW_Push, SW41 SW_Push, SW42 SW_Push, SW43 SW_Push, SW44 SW_Push, SW45 SW_Push, SW46 SW_Push, SW47 SW_Push, SW48 SW_Push, SW49 SW_Push, SW5 SW_Push, SW50 SW_Push, SW51 SW_Push, SW52 SW_Push, SW53 SW_Push, SW54 SW_Push, SW55 SW_Push, SW56 SW_Push, SW57 SW_Push, SW58 SW_Push, SW59 SW_Push, SW6 SW_Push, SW60 SW_Push, SW61 SW_Push, SW62 SW_Push, SW63 SW_Push, SW64 SW_Push, SW65 SW_Push, SW66 SW_Push, SW67 SW_Push, SW68 SW_Push, SW69 SW_Push, SW7 SW_Push, SW70 SW_Push, SW71 SW_Push, SW72 SW_Push, SW73 SW_Push, SW74 SW_Push, SW75 SW_Push, SW76 SW_Push, SW77 SW_Push, SW8 SW_Push, SW9 SW_Push, U1 ATmega16U4-AU, U2 TPD2S017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

Commit message: Updated project
Parts:
- removed C1, C2: 22p, C_0603_1608Metric
- removed C3, C4, C5, C6: 0.1u, C_0603_1608Metric
- removed C7: 4.7u, C_0603_1608Metric
- removed C8: 1u, C_0603_1608Metric
- removed D1, D10, D11, D12, D13, D14, D15, D16, D17, D18, D19, D2, D20, D21, D22, D23, D24, D25, D26, D27, D28, D29, D3, D30, D31, D32, D33, D34, D35, D36, D37, D38, D39, D4, D40, D41, D42, D43, D44, D45, D46, D47, D48, D49, D5, D50, D51, D52, D53, D54, D55, D56, D57, D58, D59, D6, D60, D61, D62, D63, D64, D65, D66, D67, D68, D69, D7, D70, D71, D72, D73, D74, D75, D76, D77, D8, D9: D, D_SOD-323F
- removed J1: USB_C_Receptacle_USB2.0, USB_C_Receptacle_XKB_U262-16XN-4BVC11
- removed R1, R2: 22, R_0603_1608Metric
- removed R3, R4: 10k, R_0603_1608Metric
- removed RST: SW_SPST, SW_SPST_TL3342
- removed ST27: MountingHole, Stabilizer_Cherry_MX_2u
- removed ST72: MountingHole, Stabilizer_Cherry_MX_6u
- removed SW1, SW10, SW11, SW12, SW13, SW14, SW15, SW16, SW17, SW18, SW19, SW2, SW20, SW21, SW22, SW23, SW24, SW25, SW26, SW29, SW3, SW30, SW31, SW32, SW33, SW34, SW35, SW36, SW37, SW38, SW39, SW4, SW40, SW43, SW44, SW45, SW46, SW47, SW48, SW49, SW5, SW50, SW51, SW52, SW53, SW54, SW56, SW57, SW58, SW59, SW6, SW60, SW61, SW62, SW63, SW64, SW65, SW66, SW67, SW68, SW7, SW74, SW75, SW76, SW77, SW8, SW9: SW_Push, SW_Cherry_MX_PCB_1.00u
- removed SW27: SW_Push, SW_Cherry_MX_PCB_2.00u
- removed SW28: SW_Push, SW_Cherry_MX_PCB_1.50u
- removed SW41: SW_Push, SW_Cherry_MX_PCB_ISOEnter
- removed SW42: SW_Push, SW_Cherry_MX_PCB_1.75u
- removed SW55, SW69, SW70, SW71, SW73: SW_Push, SW_Cherry_MX_PCB_1.25u
- removed SW72: SW_Push, SW_Cherry_MX_PCB_6.25u
- removed U1: ATmega16U4-AU, TQFP-44_10x10mm_P0.8mm
- removed U2: TPD2S017, SOT-23-6
- removed Y1: Crystal_GND24, Crystal_SMD_3225-4Pin_3.2x2.5mm
- added D_0: D, Diode_SMD:D_SOD-123, B.Cu at (18.1, 10.0)
- added D_1: D, Diode_SMD:D_SOD-123, B.Cu at (56.1, 10.0)
- added D_10: D, Diode_SMD:D_SOD-123, B.Cu at (246.7, 10.0)
- added D_11: D, Diode_SMD:D_SOD-123, B.Cu at (265.7, 10.0)
- added D_12: D, Diode_SMD:D_SOD-123, B.Cu at (284.8, 10.0)
- added D_13: D, Diode_SMD:D_SOD-123, B.Cu at (18.1, 33.8)
- added D_14: D, Diode_SMD:D_SOD-123, B.Cu at (37.1, 33.8)
- added D_15: D, Diode_SMD:D_SOD-123, B.Cu at (56.1, 33.8)
- added D_16: D, Diode_SMD:D_SOD-123, B.Cu at (75.2, 33.8)
- added D_17: D, Diode_SMD:D_SOD-123, B.Cu at (94.2, 33.8)
- added D_18: D, Diode_SMD:D_SOD-123, B.Cu at (113.3, 33.8)
- added D_19: D, Diode_SMD:D_SOD-123, B.Cu at (132.3, 33.8)
- added D_2: D, Diode_SMD:D_SOD-123, B.Cu at (75.2, 10.0)
- added D_20: D, Diode_SMD:D_SOD-123, B.Cu at (151.4, 33.8)
- added D_21: D, Diode_SMD:D_SOD-123, B.Cu at (170.4, 33.8)
- added D_22: D, Diode_SMD:D_SOD-123, B.Cu at (189.5, 33.8)
- added D_23: D, Diode_SMD:D_SOD-123, B.Cu at (208.6, 33.8)
- added D_24: D, Diode_SMD:D_SOD-123, B.Cu at (227.6, 33.8)
- added D_25: D, Diode_SMD:D_SOD-123, B.Cu at (246.7, 33.8)
- added D_26: D, Diode_SMD:D_SOD-123, B.Cu at (284.8, 33.8)
- added D_27: D, Diode_SMD:D_SOD-123, B.Cu at (27.6, 52.9)
- added D_28: D, Diode_SMD:D_SOD-123, B.Cu at (46.6, 52.9)
- added D_29: D, Diode_SMD:D_SOD-123, B.Cu at (65.7, 52.9)
- added D_3: D, Diode_SMD:D_SOD-123, B.Cu at (94.2, 10.0)
- added D_30: D, Diode_SMD:D_SOD-123, B.Cu at (84.7, 52.9)
- added D_31: D, Diode_SMD:D_SOD-123, B.Cu at (103.8, 52.9)
- added D_32: D, Diode_SMD:D_SOD-123, B.Cu at (122.8, 52.9)
- added D_33: D, Diode_SMD:D_SOD-123, B.Cu at (141.9, 52.9)
- added D_34: D, Diode_SMD:D_SOD-123, B.Cu at (160.9, 52.9)
- added D_35: D, Diode_SMD:D_SOD-123, B.Cu at (180.0, 52.9)
- added D_36: D, Diode_SMD:D_SOD-123, B.Cu at (199.0, 52.9)
- added D_37: D, Diode_SMD:D_SOD-123, B.Cu at (218.1, 52.9)
- added D_38: D, Diode_SMD:D_SOD-123, B.Cu at (237.1, 52.9)
- added D_39: D, Diode_SMD:D_SOD-123, B.Cu at (256.2, 52.9)
- added D_4: D, Diode_SMD:D_SOD-123, B.Cu at (113.3, 10.0)
- added D_40: D, Diode_SMD:D_SOD-123, B.Cu at (284.8, 62.4)
- added D_41: D, Diode_SMD:D_SOD-123, B.Cu at (32.3, 71.9)
- added D_42: D, Diode_SMD:D_SOD-123, B.Cu at (51.4, 71.9)
- added D_43: D, Diode_SMD:D_SOD-123, B.Cu at (70.4, 71.9)
- added D_44: D, Diode_SMD:D_SOD-123, B.Cu at (89.5, 71.9)
- added D_45: D, Diode_SMD:D_SOD-123, B.Cu at (108.5, 71.9)
- added D_46: D, Diode_SMD:D_SOD-123, B.Cu at (127.6, 71.9)
- added D_47: D, Diode_SMD:D_SOD-123, B.Cu at (146.6, 71.9)
- added D_48: D, Diode_SMD:D_SOD-123, B.Cu at (165.7, 71.9)
- added D_49: D, Diode_SMD:D_SOD-123, B.Cu at (184.7, 71.9)
- added D_5: D, Diode_SMD:D_SOD-123, B.Cu at (141.9, 10.0)
- added D_50: D, Diode_SMD:D_SOD-123, B.Cu at (203.8, 71.9)
- added D_51: D, Diode_SMD:D_SOD-123, B.Cu at (222.8, 71.9)
- added D_52: D, Diode_SMD:D_SOD-123, B.Cu at (241.9, 71.9)
- added D_53: D, Diode_SMD:D_SOD-123, B.Cu at (260.9, 71.9)
- added D_54: D, Diode_SMD:D_SOD-123, B.Cu at (22.8, 91.0)
- added D_55: D, Diode_SMD:D_SOD-123, B.Cu at (41.9, 91.0)
- added D_56: D, Diode_SMD:D_SOD-123, B.Cu at (60.9, 91.0)
- added D_57: D, Diode_SMD:D_SOD-123, B.Cu at (80.0, 91.0)
- added D_58: D, Diode_SMD:D_SOD-123, B.Cu at (99.0, 91.0)
- added D_59: D, Diode_SMD:D_SOD-123, B.Cu at (118.1, 91.0)
- added D_6: D, Diode_SMD:D_SOD-123, B.Cu at (160.9, 10.0)
- added D_60: D, Diode_SMD:D_SOD-123, B.Cu at (137.1, 91.0)
- added D_61: D, Diode_SMD:D_SOD-123, B.Cu at (156.2, 91.0)
- added D_62: D, Diode_SMD:D_SOD-123, B.Cu at (175.2, 91.0)
- added D_63: D, Diode_SMD:D_SOD-123, B.Cu at (194.3, 91.0)
- added D_64: D, Diode_SMD:D_SOD-123, B.Cu at (213.3, 91.0)
- added D_65: D, Diode_SMD:D_SOD-123, B.Cu at (232.4, 91.0)
- added D_66: D, Diode_SMD:D_SOD-123, B.Cu at (251.4, 91.0)
- added D_67: D, Diode_SMD:D_SOD-123, B.Cu at (270.5, 91.0)
- added D_68: D, Diode_SMD:D_SOD-123, B.Cu at (22.8, 110.0)
- added D_69: D, Diode_SMD:D_SOD-123, B.Cu at (46.6, 110.0)
- added D_7: D, Diode_SMD:D_SOD-123, B.Cu at (180.0, 10.0)
- added D_70: D, Diode_SMD:D_SOD-123, B.Cu at (70.4, 110.0)
- added D_71: D, Diode_SMD:D_SOD-123, B.Cu at (189.5, 110.0)
- added D_72: D, Diode_SMD:D_SOD-123, B.Cu at (213.3, 110.0)
- added D_73: D, Diode_SMD:D_SOD-123, B.Cu at (232.4, 110.0)
- added D_74: D, Diode_SMD:D_SOD-123, B.Cu at (251.4, 110.0)
- added D_75: D, Diode_SMD:D_SOD-123, B.Cu at (270.5, 110.0)
- added D_76: D, Diode_SMD:D_SOD-123, B.Cu at (289.5, 110.0)
- added D_8: D, Diode_SMD:D_SOD-123, B.Cu at (199.0, 10.0)
- added D_9: D, Diode_SMD:D_SOD-123, B.Cu at (227.6, 10.0)
- added K_0: KEYSW, MX_Alps_Hybrid:MX-1U-NoLED, F.Cu at (9.53, 9.53)
- added K_1: KEYSW, MX_Alps_Hybrid:MX-1U-NoLED, F.Cu at (47.6, 9.53)
- added K_10: KEYSW, MX_Alps_Hybrid:MX-1U-NoLED, F.Cu at (238.1, 9.53)
- added K_11: KEYSW, MX_Alps_Hybrid:MX-1U-NoLED, F.Cu at (257.2, 9.53)
- added K_12: KEYSW, MX_Alps_Hybrid:MX-1U-NoLED, F.Cu at (276.2, 9.53)
- added K_13: KEYSW, MX_Alps_Hybrid:MX-1U-NoLED, F.Cu at (9.53, 33.3)
- added K_14: KEYSW, MX_Alps_Hybrid:MX-1U-NoLED, F.Cu at (28.6, 33.3)
- added K_15: KEYSW, MX_Alps_Hybrid:MX-1U-NoLED, F.Cu at (47.6, 33.3)
- added K_16: KEYSW, MX_Alps_Hybrid:MX-1U-NoLED, F.Cu at (66.7, 33.3)
- added K_17: KEYSW, MX_Alps_Hybrid:MX-1U-NoLED, F.Cu at (85.7, 33.3)
- added K_18: KEYSW, MX_Alps_Hybrid:MX-1U-NoLED, F.Cu at (104.8, 33.3)
- added K_19: KEYSW, MX_Alps_Hybrid:MX-1U-NoLED, F.Cu at (123.8, 33.3)
- added K_2: KEYSW, MX_Alps_Hybrid:MX-1U-NoLED, F.Cu at (66.7, 9.53)
- added K_20: KEYSW, MX_Alps_Hybrid:MX-1U-NoLED, F.Cu at (142.9, 33.3)
- added K_21: KEYSW, MX_Alps_Hybrid:MX-1U-NoLED, F.Cu at (161.9, 33.3)
- added K_22: KEYSW, MX_Alps_Hybrid:MX-1U-NoLED, F.Cu at (181.0, 33.3)
- added K_23: KEYSW, MX_Alps_Hybrid:MX-1U-NoLED, F.Cu at (200.0, 33.3)
- added K_24: KEYSW, MX_Alps_Hybrid:MX-1U-NoLED, F.Cu at (219.1, 33.3)
- added K_25: KEYSW, MX_Alps_Hybrid:MX-1U-NoLED, F.Cu at (238.1, 33.3)
- added K_26: KEYSW, MX_Alps_Hybrid:MX-2U-NoLED, F.Cu at (266.7, 33.3)
- added K_27: KEYSW, MX_Alps_Hybrid:MX-1.5U-NoLED, F.Cu at (14.3, 52.4)
- added K_28: KEYSW, MX_Alps_Hybrid:MX-1U-NoLED, F.Cu at (38.1, 52.4)
- added K_29: KEYSW, MX_Alps_Hybrid:MX-1U-NoLED, F.Cu at (57.1, 52.4)
- added K_3: KEYSW, MX_Alps_Hybrid:MX-1U-NoLED, F.Cu at (85.7, 9.53)
- added K_30: KEYSW, MX_Alps_Hybrid:MX-1U-NoLED, F.Cu at (76.2, 52.4)
- added K_31: KEYSW, MX_Alps_Hybrid:MX-1U-NoLED, F.Cu at (95.2, 52.4)
- added K_32: KEYSW, MX_Alps_Hybrid:MX-1U-NoLED, F.Cu at (114.3, 52.4)
- added K_33: KEYSW, MX_Alps_Hybrid:MX-1U-NoLED, F.Cu at (133.3, 52.4)
- added K_34: KEYSW, MX_Alps_Hybrid:MX-1U-NoLED, F.Cu at (152.4, 52.4)
- added K_35: KEYSW, MX_Alps_Hybrid:MX-1U-NoLED, F.Cu at (171.4, 52.4)
- added K_36: KEYSW, MX_Alps_Hybrid:MX-1U-NoLED, F.Cu at (190.5, 52.4)
- added K_37: KEYSW, MX_Alps_Hybrid:MX-1U-NoLED, F.Cu at (209.6, 52.4)
- added K_38: KEYSW, MX_Alps_Hybrid:MX-1U-NoLED, F.Cu at (228.6, 52.4)
- added K_39: KEYSW, MX_Alps_Hybrid:MX-1U-NoLED, F.Cu at (247.7, 52.4)
- added K_4: KEYSW, MX_Alps_Hybrid:MX-1U-NoLED, F.Cu at (104.8, 9.53)
- added K_40: KEYSW, MX_Alps_Hybrid:MX-1.25U-NoLED, F.Cu at (273.8, 61.9)
- added K_41: KEYSW, MX_Alps_Hybrid:MX-1.75U-NoLED, F.Cu at (16.7, 71.4)
- added K_42: KEYSW, MX_Alps_Hybrid:MX-1U-NoLED, F.Cu at (42.9, 71.4)
- added K_43: KEYSW, MX_Alps_Hybrid:MX-1U-NoLED, F.Cu at (61.9, 71.4)
- added K_44: KEYSW, MX_Alps_Hybrid:MX-1U-NoLED, F.Cu at (81.0, 71.4)
- added K_45: KEYSW, MX_Alps_Hybrid:MX-1U-NoLED, F.Cu at (100.0, 71.4)
- added K_46: KEYSW, MX_Alps_Hybrid:MX-1U-NoLED, F.Cu at (119.1, 71.4)
- added K_47: KEYSW, MX_Alps_Hybrid:MX-1U-NoLED, F.Cu at (138.1, 71.4)
- added K_48: KEYSW, MX_Alps_Hybrid:MX-1U-NoLED, F.Cu at (157.2, 71.4)
- added K_49: KEYSW, MX_Alps_Hybrid:MX-1U-NoLED, F.Cu at (176.2, 71.4)
- added K_5: KEYSW, MX_Alps_Hybrid:MX-1U-NoLED, F.Cu at (133.3, 9.53)
- added K_50: KEYSW, MX_Alps_Hybrid:MX-1U-NoLED, F.Cu at (195.3, 71.4)
- added K_51: KEYSW, MX_Alps_Hybrid:MX-1U-NoLED, F.Cu at (214.3, 71.4)
- added K_52: KEYSW, MX_Alps_Hybrid:MX-1U-NoLED, F.Cu at (233.4, 71.4)
- added K_53: KEYSW, MX_Alps_Hybrid:MX-1U-NoLED, F.Cu at (252.4, 71.4)
- added K_54: KEYSW, MX_Alps_Hybrid:MX-1.25U-NoLED, F.Cu at (11.9, 90.5)
- added K_55: KEYSW, MX_Alps_Hybrid:MX-1U-NoLED, F.Cu at (33.3, 90.5)
- added K_56: KEYSW, MX_Alps_Hybrid:MX-1U-NoLED, F.Cu at (52.4, 90.5)
- added K_57: KEYSW, MX_Alps_Hybrid:MX-1U-NoLED, F.Cu at (71.4, 90.5)
- added K_58: KEYSW, MX_Alps_Hybrid:MX-1U-NoLED, F.Cu at (90.5, 90.5)
- added K_59: KEYSW, MX_Alps_Hybrid:MX-1U-NoLED, F.Cu at (109.5, 90.5)
- added K_6: KEYSW, MX_Alps_Hybrid:MX-1U-NoLED, F.Cu at (152.4, 9.53)
- added K_60: KEYSW, MX_Alps_Hybrid:MX-1U-NoLED, F.Cu at (128.6, 90.5)
- added K_61: KEYSW, MX_Alps_Hybrid:MX-1U-NoLED, F.Cu at (147.6, 90.5)
- added K_62: KEYSW, MX_Alps_Hybrid:MX-1U-NoLED, F.Cu at (166.7, 90.5)
- added K_63: KEYSW, MX_Alps_Hybrid:MX-1U-NoLED, F.Cu at (185.7, 90.5)
- added K_64: KEYSW, MX_Alps_Hybrid:MX-1U-NoLED, F.Cu at (204.8, 90.5)
- added K_65: KEYSW, MX_Alps_Hybrid:MX-1U-NoLED, F.Cu at (223.8, 90.5)
- added K_66: KEYSW, MX_Alps_Hybrid:MX-1U-NoLED, F.Cu at (242.9, 90.5)
- added K_67: KEYSW, MX_Alps_Hybrid:MX-1U-NoLED, F.Cu at (261.9, 90.5)
- added K_68: KEYSW, MX_Alps_Hybrid:MX-1.25U-NoLED, F.Cu at (11.9, 109.5)
- added K_69: KEYSW, MX_Alps_Hybrid:MX-1.25U-NoLED, F.Cu at (35.7, 109.5)
- added K_7: KEYSW, MX_Alps_Hybrid:MX-1U-NoLED, F.Cu at (171.4, 9.53)
- added K_70: KEYSW, MX_Alps_Hybrid:MX-1.25U-NoLED, F.Cu at (59.5, 109.5)
- added K_71: KEYSW, MX_Alps_Hybrid:MX-6.25U-NoLED, F.Cu at (131.0, 109.5)
- added K_72: KEYSW, MX_Alps_Hybrid:MX-1.25U-NoLED, F.Cu at (202.4, 109.5)
- added K_73: KEYSW, MX_Alps_Hybrid:MX-1U-NoLED, F.Cu at (223.8, 109.5)
- added K_74: KEYSW, MX_Alps_Hybrid:MX-1U-NoLED, F.Cu at (242.9, 109.5)
- added K_75: KEYSW, MX_Alps_Hybrid:MX-1U-NoLED, F.Cu at (261.9, 109.5)
- added K_76: KEYSW, MX_Alps_Hybrid:MX-1U-NoLED, F.Cu at (281.0, 109.5)
- added K_8: KEYSW, MX_Alps_Hybrid:MX-1U-NoLED, F.Cu at (190.5, 9.53)
- added K_9: KEYSW, MX_Alps_Hybrid:MX-1U-NoLED, F.Cu at (219.1, 9.53)
- moved ST41 35.4 mm to (273.8, 61.9)
Routing:
- net ROW5: track 269.1 -> 0.00 mm
- net ROW0: track 266.7 -> 0.00 mm
- net ROW3: track 261.2 -> 0.00 mm
- net ROW1: track 257.2 -> 0.00 mm
- net ROW4: track 250.0 -> 0.00 mm
- net ROW2: track 233.4 -> 0.00 mm
- net COL3: track 114.8 -> 0.00 mm
- net COL10: track 114.8 -> 0.00 mm
- net COL13: track 110.1 -> 0.00 mm
- net COL14: track 109.9 -> 0.00 mm
- net COL12: track 109.9 -> 0.00 mm
- net COL11: track 109.9 -> 0.00 mm
- net COL0: track 104.9 -> 0.00 mm
- net COL9: track 94.8 -> 0.00 mm
- net COL7: track 94.8 -> 0.00 mm
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Other:
- board size 295.5 x 124 mm -> 298.5 x 127.1 mm

Commit message: 1st version of PCB complete
Parts:
- removed ST41: MountingHole, Stabilizer_Cherry_MX_2u
- added C1: 22pF, Capacitor_SMD:C_0805_2012Metric, B.Cu at (87.3, 106.4)
- added C2: 22pF, Capacitor_SMD:C_0805_2012Metric, B.Cu at (87.3, 114.3)
- added C3: 1uF, Capacitor_SMD:C_0805_2012Metric, B.Cu at (99.6, 119.6)
- added C4: 0.1uF, Capacitor_SMD:C_0805_2012Metric, B.Cu at (96.0, 119.6)
- added C5: 0.1uF, Capacitor_SMD:C_0805_2012Metric, B.Cu at (95.4, 101.6)
- added C6: 0.1uF, Capacitor_SMD:C_0805_2012Metric, B.Cu at (108.0, 114.3)
- added C7: 10uF, Capacitor_SMD:C_0805_2012Metric, B.Cu at (108.0, 107.2)
- added F1: 500mA, Fuse:Fuse_1206_3216Metric, B.Cu at (23.9, 6.48)
- added R1: 10k, Resistor_SMD:R_0805_2012Metric, B.Cu at (92.2, 119.6)
- added R2: 22, Resistor_SMD:R_0805_2012Metric, B.Cu at (29.3, 6.35)
- added R3: 22, Resistor_SMD:R_0805_2012Metric, B.Cu at (27.1, 6.35)
- added R4: 10k, Resistor_SMD:R_0805_2012Metric, B.Cu at (103.2, 101.6)
- added SW1: SW_Push, random-keyboard-parts:SKQG-1155865, B.Cu at (116.7, 119.4)
- added U1: ATmega32U4-AU, Package_QFP:TQFP-44_10x10mm_P0.8mm, B.Cu at (98.4, 110.3)
- added USB1: Molex-0548190589, random-keyboard-parts:Molex-0548190589, B.Cu at (28.6, -2.38)
- added Y1: 16MHz, Crystal:Crystal_SMD_3225-4Pin_3.2x2.5mm, B.Cu at (87.3, 110.3)
- K_40: footprint MX_Alps_Hybrid:MX-1.25U-NoLED -> MX_Alps_Hybrid:MX-ISOEnter-NoLED
- moved D_71 49.3 mm to (140.2, 110.0)
Routing:
- net row0: track 0.00 -> 521.4 mm, vias 0 -> 4
- net row1: track 0.00 -> 503.9 mm, vias 0 -> 6
- net row2: track 0.00 -> 485.0 mm, vias 0 -> 6
- net row3: track 0.00 -> 433.7 mm, vias 0 -> 6
- net col13: track 0.00 -> 310.7 mm, vias 0 -> 3
- net row5: track 0.00 -> 302.4 mm, vias 0 -> 5
- net col12: track 0.00 -> 297.7 mm, vias 0 -> 1
- net col11: track 0.00 -> 295.2 mm, vias 0 -> 7
- net row4: track 0.00 -> 291.2 mm, vias 0 -> 6
- net col10: track 0.00 -> 271.3 mm, vias 0 -> 9
- net GND: track 0.00 -> 262.4 mm, vias 0 -> 2
- net col9: track 0.00 -> 247.7 mm, vias 0 -> 3
- net +5V: track 0.00 -> 218.6 mm, vias 0 -> 2
- net col0: track 0.00 -> 214.4 mm, vias 0 -> 1
- net Net-(R3-Pad1): track 0.00 -> 201.4 mm, vias 0 -> 2
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Other:
- board size 298.5 x 127.1 mm -> 298.4 x 127 mm
- net class Default: trace_width 0.25 -> 0.254
- net class Power added: clearance 0.2, trace_width 0.381, via_dia 0.8, via_drill 0.4

Commit message: Revised traces
Parts:
- added REF**: MountingHole_3.2mm_M3, MountingHole:MountingHole_3.2mm_M3, F.Cu at (0.13, 0.13)
- added REF**: MountingHole_3.2mm_M3, MountingHole:MountingHole_3.2mm_M3, F.Cu at (0.13, 119.0)
- added REF**: MountingHole_3.2mm_M3, MountingHole:MountingHole_3.2mm_M3, F.Cu at (290.4, 119.0)
- added REF**: MountingHole_3.2mm_M3, MountingHole:MountingHole_3.2mm_M3, F.Cu at (290.4, 0.13)
Connections:
- USB1 pad 6: Net-(USB1-Pad6) -> GND
Routing:
- net row2: track 485.0 -> 467.7 mm
- net Net-(USB1-Pad6): track 16.6 -> 0.00 mm
- net row3: track 433.7 -> 417.6 mm
- net GND: track 262.4 -> 276.6 mm, vias 2 -> 12
- net row1: track 503.9 -> 490.2 mm
- net row0: track 521.4 -> 508.8 mm
- net row4: track 291.2 -> 288.1 mm
- added copper zone on B.Cu, net GND
Other:
- board text added: "BareDev by ManoShu rev1"

Commit message: Added production files and added text to PCB
Parts:
- added BAREDEV_LOGO: , My:BAREDEV_LOGO, F.Cu at (273.4, 80.8)
Routing:
- net col9: track 247.7 -> 248.7 mm
Other:
- board text removed: "BareDev by ManoShu rev1"
