File: kicad_v2/keyboard.sch (KiCad schematic (older format))
At the start: 154 parts

Commit message: v2 board DRC cleared
Parts:
- added C1, C2: 22pF, Capacitor_SMD:C_0805_2012Metric, symbol Device:C_Small
- added C3: 1uF, Capacitor_SMD:C_0805_2012Metric, symbol Device:C_Small
- added C4, C5, C6: 0.1uF, Capacitor_SMD:C_0805_2012Metric, symbol Device:C_Small
- added C7: 10uF, Capacitor_SMD:C_0805_2012Metric, symbol Device:C_Small
- added F1: 500mA, Fuse:Fuse_1206_3216Metric, symbol Device:Fuse_Small
- added J1: USB_C_Receptacle, Connector_USB:USB_C_Receptacle_HRO_TYPE-C-31-M-12, symbol Connector:USB_C_Receptacle
- added R1, R6: 10k, Resistor_SMD:R_0805_2012Metric, symbol Device:R_Small
- added R2, R3: 5k1, Resistor_SMD:R_0805_2012Metric, symbol Device:R_Small
- added R4, R5: 22, Resistor_SMD:R_0805_2012Metric, symbol Device:R_Small
- added SW1: SW_Push, random-keyboard-parts.:SKQG-1155865, symbol Switch:SW_Push
- added U1: ATmega32U4-AU, Package_QFP:TQFP-44_10x10mm_P0.8mm, symbol MCU_Microchip_ATmega:ATmega32U4-AU
- added Y1: Crystal_GND24_Small, Crystal:Crystal_SMD_3225-4Pin_3.2x2.5mm, symbol Device:Crystal_GND24_Small
- D_0, D_1, D_10, D_11, D_12, D_13, D_14, D_15, D_16, D_17, D_18, D_19, D_2, D_20, D_21, D_22, D_23, D_24, D_25, D_26, D_27, D_28, D_29, D_3, D_30, D_31, D_32, D_33, D_34, D_35, D_36, D_37, D_38, D_39, D_4, D_40, D_41, D_42, D_43, D_44, D_45, D_46, D_47, D_48, D_49, D_5, D_50, D_51, D_52, D_53, D_54, D_55, D_56, D_57, D_58, D_59, D_6, D_60, D_61, D_62, D_63, D_64, D_65, D_66, D_67, D_68, D_69, D_7, D_70, D_71, D_72, D_73, D_74, D_75, D_76, D_8, D_9: symbol Device:D_Small -> keyboard-rescue:D_Small-Device
- K_40: footprint MX_Only:MXOnly-1.25U-Hotswap -> MX_Only:MXOnly-ISO-NoLED-Hotswap
Connections:
- net col0: now also U1.1 (PE6)
- net col1: now also U1.8 (PB0)
- net col10: now also U1.28 (PB4)
- net col11: now also U1.29 (PB5)
- net col12: now also U1.30 (PB6)
- net col13: now also U1.31 (PC6)
- net col14: now also U1.32 (PC7)
- net col2: now also U1.9 (PB1)
- net col3: now also U1.10 (PB2)
- net col4: now also U1.11 (PB3)
- net col5: now also U1.21 (PD3)
- net col6: now also U1.22 (PD5)
- net col7: now also U1.25 (PD4)
- net col8: now also U1.26 (PD6)
- net col9: now also U1.27 (PD7)
- net row0: now also U1.36 (PF7)
- net row1: now also U1.37 (PF6)
- net row2: now also U1.38 (PF5)
- net row3: now also U1.39 (PF4)
- net row4: now also U1.40 (PF1)
- net row5: now also U1.41 (PF0)
- new net: J1.A5 (CC1), R2.1
- new net: J1.B5 (CC2), R3.2
- new net: R1.2, SW1.2, U1.13 (~RESET)
- new net: C2.1, U1.16 (XTAL2), Y1.1
- new net: C1.1, U1.17 (XTAL1), Y1.3
- new net: R6.2, U1.33 (~HWB~/PE2)
- new net: C3.1, U1.6 (UCAP)
- new net +5V: C4.1, C5.1, C6.1, C7.1, F1.2, R1.1, U1.14 (VCC), U1.2 (UVCC), U1.24 (AVCC), U1.34 (VCC), U1.44 (AVCC), U1.7 (VBUS)
- new net D+: J1.A6 (D+), J1.B6 (D+), R4.2
- new net D+_OUT: R4.1, U1.4 (D+)
- new net D-: J1.A7 (D-), J1.B7 (D-), R5.2
- new net D-_OUT: R5.1, U1.3 (D-)
- new net GND: C1.2, C2.2, C3.2, C4.2, C5.2, C6.2, C7.2, J1.A1 (GND), J1.A12 (GND), J1.B1 (GND), J1.B12 (GND), J1.S1 (SHIELD), R2.2, R3.1, R6.1, SW1.1, U1.15 (GND), U1.23 (GND), U1.35 (GND), U1.43 (GND), U1.5 (UGND), Y1.2, Y1.4
- new net VCC: F1.1, J1.A4 (VBUS), J1.A9 (VBUS), J1.B4 (VBUS), J1.B9 (VBUS)
- no-connect marks 0 -> 15
