File: kicad_v2/keyboard.kicad_pcb (KiCad board)
At the start: 2 copper layers, 298.5 x 122.3 mm, 154 parts

Commit message: v2 board DRC cleared
Parts:
- added C1: 22pF, Capacitor_SMD:C_0805_2012Metric, B.Cu at (104.4, 94.2)
- added C2: 22pF, Capacitor_SMD:C_0805_2012Metric, B.Cu at (94.0, 94.2)
- added C3: 1uF, Capacitor_SMD:C_0805_2012Metric, B.Cu at (87.9, 106.9)
- added C4: 0.1uF, Capacitor_SMD:C_0805_2012Metric, B.Cu at (87.9, 103.1)
- added C5: 0.1uF, Capacitor_SMD:C_0805_2012Metric, B.Cu at (110.7, 100.6)
- added C6: 0.1uF, Capacitor_SMD:C_0805_2012Metric, B.Cu at (110.7, 110.7)
- added C7: 10uF, Capacitor_SMD:C_0805_2012Metric, B.Cu at (87.9, 110.7)
- added F1: 500mA, Fuse:Fuse_1206_3216Metric, B.Cu at (35.1, 7.62)
- added J1: USB_C_Receptacle, Connector_USB:USB_C_Receptacle_HRO_TYPE-C-31-M-12, B.Cu at (27.4, -1.27)
- added R1: 10k, Resistor_SMD:R_0805_2012Metric, B.Cu at (87.9, 99.3)
- added R2: 5k1, Resistor_SMD:R_0805_2012Metric, B.Cu at (23.6, 8.89)
- added R3: 5k1, Resistor_SMD:R_0805_2012Metric, B.Cu at (31.5, 8.89)
- added R4: 22, Resistor_SMD:R_0805_2012Metric, B.Cu at (28.7, 8.89)
- added R5: 22, Resistor_SMD:R_0805_2012Metric, B.Cu at (26.4, 8.89)
- added R6: 10k, Resistor_SMD:R_0805_2012Metric, B.Cu at (110.7, 105.7)
- added SW1: SW_Push, random-keyboard-parts.:SKQG-1155865, B.Cu at (285.5, 85.6)
- added U1: ATmega32U4-AU, Package_QFP:TQFP-44_10x10mm_P0.8mm, B.Cu at (99.3, 105.7)
- added Y1: Crystal_GND24_Small, Crystal:Crystal_SMD_3225-4Pin_3.2x2.5mm, B.Cu at (99.3, 94.5)
- K_40: footprint MX_Only:MXOnly-1.25U-Hotswap -> MX_Only:MXOnly-ISO-NoLED-Hotswap
- moved D_71 50.1 mm to (139.4, 105.3)
- moved D_26 9.67 mm to (275.1, 29.1)
- moved K_40 9.52 mm to (273.8, 57.1)
- moved D_40 8.89 mm to (284.8, 57.0)
Routing:
- net row0: track 0.00 -> 528.2 mm
- net row1: track 0.00 -> 498.6 mm
- net row3: track 0.00 -> 472.3 mm
- net row2: track 0.00 -> 455.2 mm
- net row4: track 0.00 -> 428.3 mm
- net row5: track 0.00 -> 308.2 mm, vias 0 -> 2
- net col14: track 0.00 -> 296.4 mm, vias 0 -> 3
- net col13: track 0.00 -> 285.6 mm, vias 0 -> 6
- net Net-(R1-Pad2): track 0.00 -> 274.2 mm, vias 0 -> 2
- net col12: track 0.00 -> 266.0 mm, vias 0 -> 7
- net col11: track 0.00 -> 247.1 mm, vias 0 -> 7
- net col10: track 0.00 -> 230.3 mm, vias 0 -> 7
- net +5V: track 0.00 -> 224.1 mm, vias 0 -> 2
- net col0: track 0.00 -> 217.8 mm, vias 0 -> 7
- net col9: track 0.00 -> 207.0 mm, vias 0 -> 6
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- added copper zone on B.Cu, net GND
Other:
- net class Power added: clearance 0.2, trace_width 0.381, via_dia 0.8, via_drill 0.4

Commit message: Added text
Other:
- board text added: "BareDev by ManoShu v2 rev1"
