File: kicad/rev2/keyboard.kicad_sch (KiCad schematic)
At the start: 255 parts, among them Q1 AO3401A, SW1 SW_Push, U1 ATmega32U4-AU, U2 USBLC6-2SC6, Y1 16MHz

Commit message: rev2 base PCB done
Parts:
- D1: footprint LED_SMD:LED_0603_1608Metric_Pad1.05x0.95mm_HandSolder -> LED_SMD:LED_0603_1608Metric
- F1: footprint Fuse:Fuse_1206_3216Metric_Pad1.42x1.75mm_HandSolder -> Fuse:Fuse_1206_3216Metric
- K_26: footprint MX_Only:MXOnly-1U -> MX_Only:MXOnly-2U-ReversedStabilizers
- K_40: footprint MX_Only:MXOnly-ISO -> My:MXOnly-ISO_NorthFacing
- K_71: footprint MX_Only:MXOnly-6.25U -> MX_Only:MXOnly-6.25U-ReversedStabilizers
- Q1: footprint Package_TO_SOT_SMD:SOT-23_Handsoldering -> Package_TO_SOT_SMD:SOT-23
- U2: footprint Package_TO_SOT_SMD:SOT-23-6_Handsoldering -> Package_TO_SOT_SMD:SOT-23-6
- USB1: footprint Type-C:HRO-TYPE-C-31-M-12-HandSoldering -> Type-C:HRO-TYPE-C-31-M-12-Assembly
Connections:
- net +5V: no longer K_0.4 (LEDGND), K_1.4 (LEDGND), K_10.4 (LEDGND), K_11.4 (LEDGND), K_12.4 (LEDGND), K_13.4 (LEDGND), K_14.4 (LEDGND), K_15.4 (LEDGND), K_16.4 (LEDGND), K_17.4 (LEDGND), K_18.4 (LEDGND), K_19.4 (LEDGND), K_2.4 (LEDGND), K_20.4 (LEDGND), K_21.4 (LEDGND), K_22.4 (LEDGND), K_23.4 (LEDGND), K_24.4 (LEDGND), K_25.4 (LEDGND), K_26.4 (LEDGND), K_27.4 (LEDGND), K_28.4 (LEDGND), K_29.4 (LEDGND), K_3.4 (LEDGND), K_30.4 (LEDGND), K_31.4 (LEDGND), K_32.4 (LEDGND), K_33.4 (LEDGND), K_34.4 (LEDGND), K_35.4 (LEDGND), K_36.4 (LEDGND), K_37.4 (LEDGND), K_38.4 (LEDGND), K_39.4 (LEDGND), K_4.4 (LEDGND), K_40.4 (LEDGND), K_41.4 (LEDGND), K_42.4 (LEDGND), K_43.4 (LEDGND), K_44.4 (LEDGND), K_45.4 (LEDGND), K_46.4 (LEDGND), K_47.4 (LEDGND), K_48.4 (LEDGND), K_49.4 (LEDGND), K_5.4 (LEDGND), K_50.4 (LEDGND), K_51.4 (LEDGND), K_52.4 (LEDGND), K_53.4 (LEDGND), K_54.4 (LEDGND), K_55.4 (LEDGND), K_56.4 (LEDGND), K_57.4 (LEDGND), K_58.4 (LEDGND), K_59.4 (LEDGND), K_6.4 (LEDGND), K_60.4 (LEDGND), K_61.4 (LEDGND), K_62.4 (LEDGND), K_63.4 (LEDGND), K_64.4 (LEDGND), K_65.4 (LEDGND), K_66.4 (LEDGND), K_67.4 (LEDGND), K_68.4 (LEDGND), K_69.4 (LEDGND), K_7.4 (LEDGND), K_70.4 (LEDGND), K_71.4 (LEDGND), K_72.4 (LEDGND), K_73.4 (LEDGND), K_74.4 (LEDGND), K_75.4 (LEDGND), K_76.4 (LEDGND), K_8.4 (LEDGND), K_9.4 (LEDGND)
- net GND: now also K_0.4 (LEDGND), K_1.4 (LEDGND), K_10.4 (LEDGND), K_11.4 (LEDGND), K_12.4 (LEDGND), K_13.4 (LEDGND), K_14.4 (LEDGND), K_15.4 (LEDGND), K_16.4 (LEDGND), K_17.4 (LEDGND), K_18.4 (LEDGND), K_19.4 (LEDGND), K_2.4 (LEDGND), K_20.4 (LEDGND), K_21.4 (LEDGND), K_22.4 (LEDGND), K_23.4 (LEDGND), K_24.4 (LEDGND), K_25.4 (LEDGND), K_26.4 (LEDGND), K_27.4 (LEDGND), K_28.4 (LEDGND), K_29.4 (LEDGND), K_3.4 (LEDGND), K_30.4 (LEDGND), K_31.4 (LEDGND), K_32.4 (LEDGND), K_33.4 (LEDGND), K_34.4 (LEDGND), K_35.4 (LEDGND), K_36.4 (LEDGND), K_37.4 (LEDGND), K_38.4 (LEDGND), K_39.4 (LEDGND), K_4.4 (LEDGND), K_40.4 (LEDGND), K_41.4 (LEDGND), K_42.4 (LEDGND), K_43.4 (LEDGND), K_44.4 (LEDGND), K_45.4 (LEDGND), K_46.4 (LEDGND), K_47.4 (LEDGND), K_48.4 (LEDGND), K_49.4 (LEDGND), K_5.4 (LEDGND), K_50.4 (LEDGND), K_51.4 (LEDGND), K_52.4 (LEDGND), K_53.4 (LEDGND), K_54.4 (LEDGND), K_55.4 (LEDGND), K_56.4 (LEDGND), K_57.4 (LEDGND), K_58.4 (LEDGND), K_59.4 (LEDGND), K_6.4 (LEDGND), K_60.4 (LEDGND), K_61.4 (LEDGND), K_62.4 (LEDGND), K_63.4 (LEDGND), K_64.4 (LEDGND), K_65.4 (LEDGND), K_66.4 (LEDGND), K_67.4 (LEDGND), K_68.4 (LEDGND), K_69.4 (LEDGND), K_7.4 (LEDGND), K_70.4 (LEDGND), K_71.4 (LEDGND), K_72.4 (LEDGND), K_73.4 (LEDGND), K_74.4 (LEDGND), K_75.4 (LEDGND), K_76.4 (LEDGND), K_8.4 (LEDGND), K_9.4 (LEDGND)
- net _RESET: now reaches R1.2, SW1.2, U1.13 (~{RESET})
- net _D-: now reaches R3.1, U1.3 (D-)
- net _D+: now reaches R2.1, U1.4 (D+)

Commit message: base rev2 PCB done
Parts:
- added H1, H2, H3, H4: MountingHole, MountingHole:MountingHole_3.2mm_M3, symbol Mechanical:MountingHole
Connections:
- net CAPS_LOCK: now also U1.41 (PF0); no longer U1.36 (PF7)
- net LEDS: now also U1.31 (PC6)
- net col1: now also U1.29 (PB5); no longer U1.12 (PB7)
- net col10: now also U1.18 (PD0); no longer U1.26 (PD6)
- net col11: now also U1.12 (PB7); no longer U1.27 (PD7)
- net col12: now also U1.11 (PB3); no longer U1.1 (PE6)
- net col13: now also U1.10 (PB2); no longer U1.41 (PF0)
- net col2: now also U1.28 (PB4); no longer U1.31 (PC6)
- net col3: now also U1.27 (PD7); no longer U1.32 (PC7)
- net col4: now also U1.26 (PD6); no longer U1.18 (PD0)
- net col5: now also U1.25 (PD4); no longer U1.19 (PD1)
- net col6: now also U1.22 (PD5); no longer U1.20 (PD2)
- net col8: now also U1.20 (PD2); no longer U1.25 (PD4)
- net col9: now also U1.19 (PD1); no longer U1.22 (PD5)
- net row0: now also U1.1 (PE6); no longer U1.8 (PB0)
- net row1: now also U1.36 (PF7); no longer U1.9 (PB1)
- net row2: now also U1.37 (PF6); no longer U1.10 (PB2)
- net row3: now also U1.38 (PF5); no longer U1.11 (PB3)
- net row4: now also U1.39 (PF4); no longer U1.28 (PB4)
- net row5: now also U1.40 (PF1); no longer U1.29 (PB5)
- no-connect marks 7 -> 5

Commit message: rev2 PCB finished
Parts:
- D1: footprint LED_SMD:LED_0603_1608Metric -> LED_SMD:LED_0603_1608Metric_Pad1.05x0.95mm_HandSolder
Changed lines of the file:
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@@
     (property "Reference" "D1" (id 0) (at 246.2022 183.7182 0))
     (property "Value" "LED" (id 1) (at 246.2022 186.0296 0))
-    (property "Footprint" "LED_SMD:LED_0603_1608Metric" (id 2) (at 246.38 189.23 0)
+    (property "Footprint" "LED_SMD:LED_0603_1608Metric_Pad1.05x0.95mm_HandSolder" (id 2) (at 246.38 189.23 0)
       (effects (font (size 1.27 1.27)) hide)
     )
@@
     )
     (path "/4bf0727d-6b56-44b6-9a02-6ac7fae46a01"
-      (reference "D1") (unit 1) (value "LED") (footprint "LED_SMD:LED_0603_1608Metric")
+      (reference "D1") (unit 1) (value "LED") (footprint "LED_SMD:LED_0603_1608Metric_Pad1.05x0.95mm_HandSolder")
     )
     (path "/d8603679-3e7b-4337-8dbc-1827f5f54d8a"

Commit message: Applied major silk screen drawings
Parts:
- C1, C2, C3, C4, C5, C6, C7: footprint Capacitor_SMD:C_0805_2012Metric -> My:C_0805_2012Metric_NoSilk
- D_0, D_1, D_10, D_11, D_12, D_13, D_14, D_15, D_16, D_17, D_18, D_19, D_2, D_20, D_21, D_22, D_23, D_24, D_25, D_26, D_27, D_28, D_29, D_3, D_30, D_31, D_32, D_33, D_34, D_35, D_36, D_37, D_38, D_39, D_4, D_40, D_41, D_42, D_43, D_44, D_45, D_46, D_47, D_48, D_49, D_5, D_50, D_51, D_52, D_53, D_54, D_55, D_56, D_57, D_58, D_59, D_6, D_60, D_61, D_62, D_63, D_64, D_65, D_66, D_67, D_68, D_69, D_7, D_70, D_71, D_72, D_73, D_74, D_75, D_76, D_8, D_9: footprint Diode_SMD:D_SOD-123 -> My:D_SOD-123_NoSilk
- R1, R10, R11, R12, R13, R14, R15, R16, R17, R18, R19, R2, R20, R21, R22, R23, R24, R25, R26, R27, R28, R29, R3, R30, R31, R32, R33, R34, R35, R36, R37, R38, R39, R4, R40, R41, R42, R43, R44, R45, R46, R47, R48, R49, R5, R50, R51, R52, R53, R54, R55, R56, R57, R58, R59, R6, R60, R61, R62, R63, R64, R65, R66, R67, R68, R69, R7, R70, R71, R72, R73, R74, R75, R76, R77, R78, R79, R8, R80, R81, R82, R83, R84, R85, R86, R9: footprint Resistor_SMD:R_0805_2012Metric -> My:R_0805_2012Metric_NoSilk
