File: kicad/rev2b/BareDevRev2.kicad_sch (KiCad schematic)
At the start: 19 parts, among them U1 BL24C256A-SFRC, U2 JOKER MCU, X1 ARM JTAG, Y1 7325-0800A2010-00

Commit message: Updated .gitmodules (???)
Parts:
- added D_? (x77): D, My:D_SOD-123_NoSilk, symbol Device:D_Small
- added K_? (x67): KEYSW, MX_Only:MXOnly-1U, symbol MX_Alps_Hybrid:MX-LED
- added K_? (x5): KEYSW, MX_Only:MXOnly-1.25U, symbol MX_Alps_Hybrid:MX-LED
- added K_?: KEYSW, MX_Only:MXOnly-1.5U, symbol MX_Alps_Hybrid:MX-LED
- added K_?: KEYSW, My:MXOnly-ISO_NorthFacing, symbol MX_Alps_Hybrid:MX-LED
- added K_?: KEYSW, MX_Only:MXOnly-1.75U, symbol MX_Alps_Hybrid:MX-LED
- added K_?: KEYSW, MX_Only:MXOnly-2U-ReversedStabilizers, symbol MX_Alps_Hybrid:MX-LED
- added K_?: KEYSW, MX_Only:MXOnly-6.25U-ReversedStabilizers, symbol MX_Alps_Hybrid:MX-LED
- added R? (x77): 2K, My:R_0805_2012Metric_NoSilk, symbol Device:R_Small
Connections:
- net GND: now also K_?.4 (LEDGND), K_?.4 (LEDGND), K_?.4 (LEDGND), K_?.4 (LEDGND), K_?.4 (LEDGND), K_?.4 (LEDGND), K_?.4 (LEDGND), K_?.4 (LEDGND), K_?.4 (LEDGND), K_?.4 (LEDGND), K_?.4 (LEDGND), K_?.4 (LEDGND), K_?.4 (LEDGND), K_?.4 (LEDGND), K_?.4 (LEDGND), K_?.4 (LEDGND), K_?.4 (LEDGND), K_?.4 (LEDGND), K_?.4 (LEDGND), K_?.4 (LEDGND), K_?.4 (LEDGND), K_?.4 (LEDGND), K_?.4 (LEDGND), K_?.4 (LEDGND), K_?.4 (LEDGND), K_?.4 (LEDGND), K_?.4 (LEDGND), K_?.4 (LEDGND), K_?.4 (LEDGND), K_?.4 (LEDGND), K_?.4 (LEDGND), K_?.4 (LEDGND), K_?.4 (LEDGND), K_?.4 (LEDGND), K_?.4 (LEDGND), K_?.4 (LEDGND), K_?.4 (LEDGND), K_?.4 (LEDGND), K_?.4 (LEDGND), K_?.4 (LEDGND), K_?.4 (LEDGND), K_?.4 (LEDGND), K_?.4 (LEDGND), K_?.4 (LEDGND), K_?.4 (LEDGND), K_?.4 (LEDGND), K_?.4 (LEDGND), K_?.4 (LEDGND), K_?.4 (LEDGND), K_?.4 (LEDGND), K_?.4 (LEDGND), K_?.4 (LEDGND), K_?.4 (LEDGND), K_?.4 (LEDGND), K_?.4 (LEDGND), K_?.4 (LEDGND), K_?.4 (LEDGND), K_?.4 (LEDGND), K_?.4 (LEDGND), K_?.4 (LEDGND), K_?.4 (LEDGND), K_?.4 (LEDGND), K_?.4 (LEDGND), K_?.4 (LEDGND), K_?.4 (LEDGND), K_?.4 (LEDGND), K_?.4 (LEDGND), K_?.4 (LEDGND), K_?.4 (LEDGND), K_?.4 (LEDGND), K_?.4 (LEDGND), K_?.4 (LEDGND), K_?.4 (LEDGND), K_?.4 (LEDGND), K_?.4 (LEDGND), K_?.4 (LEDGND), K_?.4 (LEDGND)
- new net: D_?.2 (A), K_?.2 (ROW) (x77)
- new net: K_?.3 (LED), R?.1 (x77)
- new net COL0: K_?.1 (COL), K_?.1 (COL), K_?.1 (COL), K_?.1 (COL), K_?.1 (COL), K_?.1 (COL)
- new net COL1: K_?.1 (COL), K_?.1 (COL), K_?.1 (COL), K_?.1 (COL), K_?.1 (COL)
- new net COL10: K_?.1 (COL), K_?.1 (COL), K_?.1 (COL), K_?.1 (COL), K_?.1 (COL), K_?.1 (COL)
- new net COL11: K_?.1 (COL), K_?.1 (COL), K_?.1 (COL), K_?.1 (COL), K_?.1 (COL), K_?.1 (COL)
- new net COL12: K_?.1 (COL), K_?.1 (COL), K_?.1 (COL), K_?.1 (COL), K_?.1 (COL), K_?.1 (COL)
- new net COL13: K_?.1 (COL), K_?.1 (COL), K_?.1 (COL), K_?.1 (COL), K_?.1 (COL)
- new net COL2: K_?.1 (COL), K_?.1 (COL), K_?.1 (COL), K_?.1 (COL), K_?.1 (COL), K_?.1 (COL)
- new net COL3: K_?.1 (COL), K_?.1 (COL), K_?.1 (COL), K_?.1 (COL), K_?.1 (COL)
- new net COL4: K_?.1 (COL), K_?.1 (COL), K_?.1 (COL), K_?.1 (COL), K_?.1 (COL)
- new net COL5: K_?.1 (COL), K_?.1 (COL), K_?.1 (COL), K_?.1 (COL), K_?.1 (COL)
- new net COL6: K_?.1 (COL), K_?.1 (COL), K_?.1 (COL), K_?.1 (COL), K_?.1 (COL), K_?.1 (COL)
- new net COL7: K_?.1 (COL), K_?.1 (COL), K_?.1 (COL), K_?.1 (COL), K_?.1 (COL)
- new net COL8: K_?.1 (COL), K_?.1 (COL), K_?.1 (COL), K_?.1 (COL), K_?.1 (COL)
- new net COL9: K_?.1 (COL), K_?.1 (COL), K_?.1 (COL), K_?.1 (COL), K_?.1 (COL), K_?.1 (COL)
- new net LED_OUT: R?.2, R?.2, R?.2, R?.2, R?.2, R?.2, R?.2, R?.2, R?.2, R?.2, R?.2, R?.2, R?.2, R?.2, R?.2, R?.2, R?.2, R?.2, R?.2, R?.2, R?.2, R?.2, R?.2, R?.2, R?.2, R?.2, R?.2, R?.2, R?.2, R?.2, R?.2, R?.2, R?.2, R?.2, R?.2, R?.2, R?.2, R?.2, R?.2, R?.2, R?.2, R?.2, R?.2, R?.2, R?.2, R?.2, R?.2, R?.2, R?.2, R?.2, R?.2, R?.2, R?.2, R?.2, R?.2, R?.2, R?.2, R?.2, R?.2, R?.2, R?.2, R?.2, R?.2, R?.2, R?.2, R?.2, R?.2, R?.2, R?.2, R?.2, R?.2, R?.2, R?.2, R?.2, R?.2, R?.2, R?.2
- new net ROW0: D_?.1 (K), D_?.1 (K), D_?.1 (K), D_?.1 (K), D_?.1 (K), D_?.1 (K), D_?.1 (K), D_?.1 (K), D_?.1 (K), D_?.1 (K), D_?.1 (K), D_?.1 (K), D_?.1 (K)
- new net ROW1: D_?.1 (K), D_?.1 (K), D_?.1 (K), D_?.1 (K), D_?.1 (K), D_?.1 (K), D_?.1 (K), D_?.1 (K), D_?.1 (K), D_?.1 (K), D_?.1 (K), D_?.1 (K), D_?.1 (K), D_?.1 (K)
- new net ROW2: D_?.1 (K), D_?.1 (K), D_?.1 (K), D_?.1 (K), D_?.1 (K), D_?.1 (K), D_?.1 (K), D_?.1 (K), D_?.1 (K), D_?.1 (K), D_?.1 (K), D_?.1 (K), D_?.1 (K), D_?.1 (K)
- new net ROW3: D_?.1 (K), D_?.1 (K), D_?.1 (K), D_?.1 (K), D_?.1 (K), D_?.1 (K), D_?.1 (K), D_?.1 (K), D_?.1 (K), D_?.1 (K), D_?.1 (K), D_?.1 (K), D_?.1 (K)
- new net ROW4: D_?.1 (K), D_?.1 (K), D_?.1 (K), D_?.1 (K), D_?.1 (K), D_?.1 (K), D_?.1 (K), D_?.1 (K), D_?.1 (K), D_?.1 (K), D_?.1 (K), D_?.1 (K), D_?.1 (K), D_?.1 (K)
- new net ROW5: D_?.1 (K), D_?.1 (K), D_?.1 (K), D_?.1 (K), D_?.1 (K), D_?.1 (K), D_?.1 (K), D_?.1 (K), D_?.1 (K)
Other:
- note added: "SWITCH MATRIX"
