File: kicad/rev2b/BareDevRev2.kicad_sch (KiCad schematic)
At the start: 250 parts, among them U1 BL24C256A-SFRC, U2 JOKER MCU, X1 ARM JTAG, Y1 7325-0800A2010-00

Commit message: initial rev2b schematic
Parts:
- added C201, C202: 1u, Capacitor_SMD:C_0805_2012Metric, symbol Device:C
- added C203: 10n, Capacitor_SMD:C_0402_1005Metric, symbol Device:C_Small
- added C301: 10u, Capacitor_SMD:C_0402_1005Metric, symbol Device:C_Small
- added C302: 100n, Capacitor_SMD:C_0402_1005Metric, symbol Device:C_Small
- added D201: B5819W-SL, acheron_Components:D_SOD-123, symbol Device:D_Schottky
- added D301: 1N4148W, acheron_Components:D_SOD-123, symbol Device:D
- added D501: LED, LED_SMD:LED_0603_1608Metric_Pad1.05x0.95mm_HandSolder, symbol Device:LED
- added F201: nSMD100-16V, Fuse:Fuse_1206_3216Metric, symbol Device:Fuse
- added FB401: GZ2012D601TF, Inductor_SMD:L_0805_2012Metric, symbol Device:FerriteBead_Small
- added J401: TYPE-C-31-M12, acheron_Connectors:USB_C_Receptacle_Hroparts_TYPE-C-31-M-12, symbol acheron_Symbols:TYPE-C-31-M-12
- added Q301, Q302: 2N7002, Package_TO_SOT_SMD:SOT-23, symbol Transistor_FET:2N7002
- added Q501: AO3401A, Package_TO_SOT_SMD:SOT-23, symbol Transistor_FET:AO3401A
- added R201, R202: 100k, Resistor_SMD:R_0805_2012Metric, symbol Device:R
- added R301: 330k, Resistor_SMD:R_0402_1005Metric, symbol Device:R_Small
- added R302: 1M, Resistor_SMD:R_0402_1005Metric, symbol Device:R_Small
- added R303, R307: 10k, Resistor_SMD:R_0402_1005Metric, symbol Device:R_Small
- added R304, R305, R306: 100R, Resistor_SMD:R_0402_1005Metric, symbol Device:R_Small
- added R308, R503: 10k, Resistor_SMD:R_0805_2012Metric, symbol Device:R_Small
- added R401, R402: 5.1k, Resistor_SMD:R_0402_1005Metric, symbol Device:R_Small
- added R501: 100, Resistor_SMD:R_0805_2012Metric, symbol Device:R_Small
- added R502: 470, Resistor_SMD:R_0805_2012Metric, symbol Device:R_Small
- added SW301: K2-1187SQ-A4SW-06, acheron_Hardware:K2-1187SQ-A4SW-06, symbol Switch:SW_SPST
- added U201: SGM2007-3.3XN5/TR, acheron_Components:SOT-23-5, symbol acheron_Symbols:SGM2036
- added U3: USBLC6-2SC6, acheron_Components:SOT-23-6, symbol Power_Protection:USBLC6-2SC6
- C5: symbol Device:CP1 -> Device:C_Polarized_US
- D_101, D_102, D_103, D_104, D_105, D_106, D_107, D_108, D_109, D_110, D_111, D_112, D_113, D_114, D_115, D_116, D_117, D_118, D_119, D_120, D_121, D_122, D_123, D_124, D_125, D_126, D_127, D_128, D_129, D_130, D_131, D_132, D_133, D_134, D_135, D_136, D_137, D_138, D_139, D_140, D_141, D_142, D_143, D_144, D_145, D_146, D_147, D_148, D_149, D_150, D_151, D_152, D_153, D_154, D_155, D_156, D_157, D_158, D_159, D_160, D_161, D_162, D_163, D_164, D_165, D_166, D_167, D_168, D_169, D_170, D_171, D_172, D_173, D_174, D_175, D_176, D_177: renamed from D_?; footprint My:D_SOD-123_NoSilk -> acheron_Components:D_SOD-123
- K_101, K_102, K_103, K_104, K_105, K_106, K_107, K_108, K_109, K_110, K_111, K_112, K_113, K_114, K_115, K_116, K_117, K_118, K_119, K_120, K_121, K_122, K_123, K_124, K_125, K_126, K_129, K_130, K_131, K_132, K_133, K_134, K_135, K_136, K_137, K_138, K_139, K_140, K_143, K_144, K_145, K_146, K_147, K_148, K_149, K_150, K_151, K_152, K_153, K_154, K_156, K_157, K_158, K_159, K_160, K_161, K_162, K_163, K_164, K_165, K_166, K_167, K_168, K_174, K_175, K_176, K_177: renamed from K_?; footprint MX_Only:MXOnly-1U -> acheron_MX_soldermask:MX100
- K_127: renamed from K_?; footprint MX_Only:MXOnly-2U-ReversedStabilizers -> acheron_MX_soldermask:MX200R
- K_128: renamed from K_?; footprint MX_Only:MXOnly-1.5U -> acheron_MX_soldermask:MX150
- K_141: renamed from K_?; footprint My:MXOnly-ISO_NorthFacing -> acheron_MX_soldermask:MX_ISOEnter_LED
- K_142: renamed from K_?; footprint MX_Only:MXOnly-1.75U -> acheron_MX_soldermask:MX175
- K_155, K_169, K_170, K_171, K_173: renamed from K_?; footprint MX_Only:MXOnly-1.25U -> acheron_MX_soldermask:MX125
- K_172: renamed from K_?; footprint MX_Only:MXOnly-6.25U-ReversedStabilizers -> acheron_MX_soldermask:MX625R
- R101, R102, R103, R104, R105, R106, R107, R108, R109, R110, R111, R112, R113, R114, R115, R116, R117, R118, R119, R120, R121, R122, R123, R124, R125, R126, R127, R128, R129, R130, R131, R132, R133, R134, R135, R136, R137, R138, R139, R140, R141, R142, R143, R144, R145, R146, R147, R148, R149, R150, R151, R152, R153, R154, R155, R156, R157, R158, R159, R160, R161, R162, R163, R164, R165, R166, R167, R168, R169, R170, R171, R172, R173, R174, R175, R176, R177: renamed from R?; footprint My:R_0805_2012Metric_NoSilk -> Resistor_SMD:R_0805_2012Metric
- U2: footprint acheron_Components:STM_UFQFPN-48_LQFP-48-1EP_7x7mm_P0.5mm_HandSoldering_ThermalReliefs -> acheron_Components:LQFP-48_7x7mm_P0.5mm; symbol acheron_Symbols:STM32F411-48 -> acheron_Symbols:STM32F411-UFQFPN48; Manufacturer (none) -> STMicroelectronics; Manufacturer Part Number (none) -> STM32F411; Package (none) -> UFQFPN-48
Connections:
- net 3V3: now also C202.1, D201.2 (A), R202.1, SW301.1 (A), U201.5 (OUT)
- net BOOT0: now also C301.1, R301.1, R302.1, R303.2
- net CAPS_INDICATOR: now also D501.2 (A)
- net COL0: now also U2.10 (PA0-WKUP), U2.11 (PA1), U2.12 (PA2), U2.13 (PA3), U2.14 (PA4), U2.15 (PA5), U2.17 (PA7), U2.18 (PB0), U2.2 (PC13), U2.21 (B10), U2.25 (PB12), U2.27 (PB14), U2.3 (PC14_OSC32IN), U2.4 (PC15_OSC32OUT)
- net D+: now also U3.3 (I/O2)
- net D-: now also U3.1 (I/O1)
- net GND: now also C201.2, C202.2, C203.1, C301.2, C302.2, FB401.1, J401.A1 (GND), J401.B1 (GND), Q301.2 (S), Q302.2 (S), R201.2, R202.2, R302.2, R307.1, R308.2, R401.1, R402.2, R502.2, U201.2 (GND), U3.2 (GND)
- net LED_OUT: now also Q501.3 (D)
- net LED_PWM: now also R501.2, R503.1
- net NRST: now also C302.1, R305.2
- net PB2/BOOT1: now also R308.1
- net ROW0: now also U2.46 (PB9)
- net ROW1: now also U2.45 (PB8)
- net ROW2: now also U2.41 (PB5)
- net ROW3: now also U2.40 (PB4)
- net ROW4: now also U2.39 (PB3)
- net ROW5: now also U2.38 (PA15)
- net PA9: no longer names the net of U2.30 (PA9)
- net PB13: no longer names the net of U2.26 (PB13)
- net RGB_3V3: no longer names the net of U2.28 (PB15)
- new net: Q301.1 (G), R304.2
- new net: Q301.3 (D), R303.1
- new net: C203.2, U201.4 (BP/FB)
- new net: D501.1 (K), R502.1
- new net: Q501.1 (G), R501.1
- new net: D301.1 (K), R301.2
- new net: D301.2 (A), R306.2, SW301.2 (B)
- new net: J401.B5 (CC2), R402.1
- new net: J401.A5 (CC1), R401.2
- new net: Q302.3 (D), R304.1, R305.1
- new net: Q302.1 (G), R306.1, R307.2
- new net 5V: C201.1, D201.1 (K), F201.1, Q501.2 (S), R201.1, R503.2, U201.1 (IN), U201.3 (EN)
- new net DBUS+: J401.A6 (D+), J401.B6 (D+), U3.4 (I/O2)
- new net DBUS-: J401.A7 (D-), J401.B7 (D-), U3.6 (I/O1)
- new net GNDPWR: FB401.2, J401.S1 (SHIELD)
- new net VBUS: F201.2, J401.A4 (VBUS), J401.B4 (VBUS), U3.5 (VBUS)
- no-connect marks 0 -> 8
Other:
- note added: "3V3"
- note added: "HARD RESET"
- note added: "USB Connector"
- note added: "USB ESD"

Commit message: Refactored matrix and LED grids
Parts:
- removed D501: LED, LED_SMD:LED_0603_1608Metric_Pad1.05x0.95mm_HandSolder, symbol Device:LED
- removed D_101, D_102, D_103, D_104, D_105, D_106, D_107, D_108, D_109, D_110, D_111, D_112, D_113, D_114, D_115, D_116, D_117, D_118, D_119, D_120, D_121, D_122, D_123, D_124, D_125, D_126, D_127, D_128, D_129, D_130, D_131, D_132, D_133, D_134, D_135, D_136, D_137, D_138, D_139, D_140, D_141, D_142, D_143, D_144, D_145, D_146, D_147, D_148, D_149, D_150, D_151, D_152, D_153, D_154, D_155, D_156, D_157, D_158, D_159, D_160, D_161, D_162, D_163, D_164, D_165, D_166, D_167, D_168, D_169, D_170, D_171, D_172, D_173, D_174, D_175, D_176, D_177: D, acheron_Components:D_SOD-123, symbol Device:D_Small
- removed K_101, K_102, K_103, K_104, K_105, K_106, K_107, K_108, K_109, K_110, K_111, K_112, K_113, K_114, K_115, K_116, K_117, K_118, K_119, K_120, K_121, K_122, K_123, K_124, K_125, K_126, K_129, K_130, K_131, K_132, K_133, K_134, K_135, K_136, K_137, K_138, K_139, K_140, K_143, K_144, K_145, K_146, K_147, K_148, K_149, K_150, K_151, K_152, K_153, K_154, K_156, K_157, K_158, K_159, K_160, K_161, K_162, K_163, K_164, K_165, K_166, K_167, K_168, K_174, K_175, K_176, K_177: KEYSW, acheron_MX_soldermask:MX100, symbol MX_Alps_Hybrid:MX-LED
- removed K_127: KEYSW, acheron_MX_soldermask:MX200R, symbol MX_Alps_Hybrid:MX-LED
- removed K_128: KEYSW, acheron_MX_soldermask:MX150, symbol MX_Alps_Hybrid:MX-LED
- removed K_141: KEYSW, acheron_MX_soldermask:MX_ISOEnter_LED, symbol MX_Alps_Hybrid:MX-LED
- removed K_142: KEYSW, acheron_MX_soldermask:MX175, symbol MX_Alps_Hybrid:MX-LED
- removed K_155, K_169, K_170, K_171, K_173: KEYSW, acheron_MX_soldermask:MX125, symbol MX_Alps_Hybrid:MX-LED
- removed K_172: KEYSW, acheron_MX_soldermask:MX625R, symbol MX_Alps_Hybrid:MX-LED
- removed Q501: AO3401A, Package_TO_SOT_SMD:SOT-23, symbol Transistor_FET:AO3401A
- removed R501: 100, Resistor_SMD:R_0805_2012Metric, symbol Device:R_Small
- removed R502: 470, Resistor_SMD:R_0805_2012Metric, symbol Device:R_Small
- removed R503: 10k, Resistor_SMD:R_0805_2012Metric, symbol Device:R_Small
- added D_101, D_102, D_103, D_104, D_105, D_106, D_107, D_108, D_109, D_110, D_111, D_112, D_113, D_114, D_115, D_116, D_117, D_118, D_119, D_120, D_121, D_122, D_123, D_124, D_125, D_126, D_127, D_128, D_129, D_130, D_131, D_132, D_133, D_134, D_135, D_136, D_137, D_138, D_139, D_140, D_141, D_142, D_143, D_144, D_145, D_146, D_147, D_148, D_149, D_150, D_151, D_152, D_153, D_154, D_155, D_156, D_157, D_158, D_159, D_160, D_161, D_162, D_163, D_164, D_165, D_166, D_167, D_168, D_169, D_170, D_171, D_172, D_173, D_174, D_175, D_176, D_177: D, acheron_Components:D_SOD-123, symbol Device:D
- added K_101, K_102, K_103, K_104, K_105, K_106, K_107, K_108, K_109, K_110, K_111, K_112, K_113, K_114, K_115, K_116, K_117, K_118, K_119, K_120, K_121, K_122, K_123, K_124, K_125, K_126, K_129, K_130, K_131, K_132, K_133, K_134, K_135, K_136, K_137, K_138, K_139, K_140, K_143, K_144, K_145, K_146, K_147, K_148, K_149, K_150, K_151, K_152, K_153, K_154, K_156, K_157, K_158, K_159, K_160, K_161, K_162, K_163, K_164, K_165, K_166, K_167, K_168, K_174, K_175, K_176, K_177: Mechanical_Switch, acheron_MX_soldermask:MX100, symbol acheron_Symbols:Mechanical_Switch
- added K_127: Mechanical_Switch, acheron_MX_soldermask:MX200, symbol acheron_Symbols:Mechanical_Switch
- added K_128: Mechanical_Switch, acheron_MX_soldermask:MX150, symbol acheron_Symbols:Mechanical_Switch
- added K_141: Mechanical_Switch, acheron_MX_soldermask:MX_ISOEnter, symbol acheron_Symbols:Mechanical_Switch
- added K_142: Mechanical_Switch, acheron_MX_soldermask:MX175, symbol acheron_Symbols:Mechanical_Switch
- added K_155, K_169, K_170, K_171, K_173: Mechanical_Switch, acheron_MX_soldermask:MX125, symbol acheron_Symbols:Mechanical_Switch
- added K_172: Mechanical_Switch, acheron_MX_soldermask:MX625, symbol acheron_Symbols:Mechanical_Switch
- added LED1, LED101, LED102, LED103, LED104, LED105, LED106, LED107, LED108, LED109, LED110, LED111, LED112, LED113, LED114, LED115, LED116, LED117, LED118, LED119, LED120, LED121, LED122, LED123, LED124, LED125, LED126, LED127, LED128, LED129, LED130, LED131, LED132, LED133, LED134, LED135, LED136, LED137, LED138, LED139, LED140, LED141, LED142, LED143, LED144, LED145, LED146, LED147, LED148, LED149, LED150, LED151, LED152, LED153, LED154, LED155, LED156, LED157, LED158, LED159, LED160, LED161, LED162, LED163, LED164, LED165, LED166, LED167, LED168, LED169, LED170, LED171, LED172, LED173, LED174, LED175, LED176, LED177: LED, acheron_Components:LED_THT_2.54mm, symbol acheron_Symbols:LED
- added Q1: AO3401A, Package_TO_SOT_SMD:SOT-23, symbol Transistor_FET:AO3401A
- added R5: 100, Resistor_SMD:R_0805_2012Metric, symbol Device:R_Small
- added R6: 10k, Resistor_SMD:R_0805_2012Metric, symbol Device:R_Small
- added R7: 470, Resistor_SMD:R_0805_2012Metric, symbol Device:R_Small
- R101, R102, R103, R104, R105, R106, R107, R108, R109, R110, R111, R112, R113, R114, R115, R116, R117, R118, R119, R120, R121, R122, R123, R124, R125, R126, R127, R128, R129, R130, R131, R132, R133, R134, R135, R136, R137, R138, R139, R140, R141, R142, R143, R144, R145, R146, R147, R148, R149, R150, R151, R152, R153, R154, R155, R156, R157, R158, R159, R160, R161, R162, R163, R164, R165, R166, R167, R168, R169, R170, R171, R172, R173, R174, R175, R176, R177: value 2K -> 2k; Manufacturer (none) -> Uniroyal; Manufacturer Part Number (none) -> 0805W8F1001T5E; Package (none) -> R0805; Specification (none) -> ±1% 125mW Thick Film Resistors 150V 0805; Vendor Part Number (none) -> LCSC C17513
Connections:
- net 5V: now also Q1.2 (S), R6.2
- net CAPS_INDICATOR: now also LED1.A
- net COL0: now also K_101.1, K_114.1, K_128.1, K_142.1, K_155.1, K_169.1
- net COL1: now also K_115.1, K_129.1, K_143.1, K_156.1, K_170.1
- net COL10: now also K_110.1, K_124.1, K_138.1, K_152.1, K_165.1, K_174.1
- net COL11: now also K_111.1, K_125.1, K_139.1, K_153.1, K_166.1, K_175.1
- net COL12: now also K_112.1, K_126.1, K_140.1, K_154.1, K_167.1, K_176.1
- net COL13: now also K_113.1, K_127.1, K_141.1, K_168.1, K_177.1
- net COL2: now also K_102.1, K_116.1, K_130.1, K_144.1, K_157.1, K_171.1
- net COL3: now also K_103.1, K_117.1, K_131.1, K_145.1, K_158.1
- net COL4: now also K_104.1, K_118.1, K_132.1, K_146.1, K_159.1
- net COL5: now also K_105.1, K_119.1, K_133.1, K_147.1, K_160.1
- net COL6: now also K_106.1, K_120.1, K_134.1, K_148.1, K_161.1, K_172.1
- net COL7: now also K_107.1, K_121.1, K_135.1, K_149.1, K_162.1
- net COL8: now also K_108.1, K_122.1, K_136.1, K_150.1, K_163.1
- net COL9: now also K_109.1, K_123.1, K_137.1, K_151.1, K_164.1, K_173.1
- net GND: now also LED101.K, LED102.K, LED103.K, LED104.K, LED105.K, LED106.K, LED107.K, LED108.K, LED109.K, LED110.K, LED111.K, LED112.K, LED113.K, LED114.K, LED115.K, LED116.K, LED117.K, LED118.K, LED119.K, LED120.K, LED121.K, LED122.K, LED123.K, LED124.K, LED125.K, LED126.K, LED127.K, LED128.K, LED129.K, LED130.K, LED131.K, LED132.K, LED133.K, LED134.K, LED135.K, LED136.K, LED137.K, LED138.K, LED139.K, LED140.K, LED141.K, LED142.K, LED143.K, LED144.K, LED145.K, LED146.K, LED147.K, LED148.K, LED149.K, LED150.K, LED151.K, LED152.K, LED153.K, LED154.K, LED155.K, LED156.K, LED157.K, LED158.K, LED159.K, LED160.K, LED161.K, LED162.K, LED163.K, LED164.K, LED165.K, LED166.K, LED167.K, LED168.K, LED169.K, LED170.K, LED171.K, LED172.K, LED173.K, LED174.K, LED175.K, LED176.K, LED177.K, R7.2
- net LED_PWM: now also R5.2, R6.1
- net ROW0: now also D_101.1 (K), D_102.1 (K), D_103.1 (K), D_104.1 (K), D_105.1 (K), D_106.1 (K), D_107.1 (K), D_108.1 (K), D_109.1 (K), D_110.1 (K), D_111.1 (K), D_112.1 (K), D_113.1 (K)
- net ROW1: now also D_114.1 (K), D_115.1 (K), D_116.1 (K), D_117.1 (K), D_118.1 (K), D_119.1 (K), D_120.1 (K), D_121.1 (K), D_122.1 (K), D_123.1 (K), D_124.1 (K), D_125.1 (K), D_126.1 (K), D_127.1 (K)
- net ROW2: now also D_128.1 (K), D_129.1 (K), D_130.1 (K), D_131.1 (K), D_132.1 (K), D_133.1 (K), D_134.1 (K), D_135.1 (K), D_136.1 (K), D_137.1 (K), D_138.1 (K), D_139.1 (K), D_140.1 (K), D_141.1 (K)
- net ROW3: now also D_142.1 (K), D_143.1 (K), D_144.1 (K), D_145.1 (K), D_146.1 (K), D_147.1 (K), D_148.1 (K), D_149.1 (K), D_150.1 (K), D_151.1 (K), D_152.1 (K), D_153.1 (K), D_154.1 (K)
- net ROW4: now also D_155.1 (K), D_156.1 (K), D_157.1 (K), D_158.1 (K), D_159.1 (K), D_160.1 (K), D_161.1 (K), D_162.1 (K), D_163.1 (K), D_164.1 (K), D_165.1 (K), D_166.1 (K), D_167.1 (K), D_168.1 (K)
- net ROW5: now also D_169.1 (K), D_170.1 (K), D_171.1 (K), D_172.1 (K), D_173.1 (K), D_174.1 (K), D_175.1 (K), D_176.1 (K), D_177.1 (K)
- net at R110.1: now also R101.1, R102.1, R103.1, R104.1, R105.1, R106.1, R107.1, R108.1, R109.1, R111.1, R112.1, R113.1, R114.1, R115.1, R116.1, R117.1, R118.1, R119.1, R120.1, R121.1, R122.1, R123.1, R124.1, R125.1, R126.1, R127.1, R128.1, R129.1, R130.1, R131.1, R132.1, R133.1, R134.1, R135.1, R136.1, R137.1, R138.1, R139.1, R140.1, R141.1, R142.1, R143.1, R144.1, R145.1, R146.1, R147.1, R148.1, R149.1, R150.1, R151.1, R152.1, R153.1, R154.1, R155.1, R156.1, R157.1, R158.1, R159.1, R160.1, R161.1, R162.1, R163.1, R164.1, R165.1, R166.1, R167.1, R168.1, R169.1, R170.1, R171.1, R172.1, R173.1, R174.1, R175.1, R176.1, R177.1, Q1.3 (D)
- removed net LED_OUT: R101.2, R102.2, R103.2, R104.2, R105.2, R106.2, R107.2, R108.2, R109.2, R110.2, R111.2, R112.2, R113.2, R114.2, R115.2, R116.2, R117.2, R118.2, R119.2, R120.2, R121.2, R122.2, R123.2, R124.2, R125.2, R126.2, R127.2, R128.2, R129.2, R130.2, R131.2, R132.2, R133.2, R134.2, R135.2, R136.2, R137.2, R138.2, R139.2, R140.2, R141.2, R142.2, R143.2, R144.2, R145.2, R146.2, R147.2, R148.2, R149.2, R150.2, R151.2, R152.2, R153.2, R154.2, R155.2, R156.2, R157.2, R158.2, R159.2, R160.2, R161.2, R162.2, R163.2, R164.2, R165.2, R166.2, R167.2, R168.2, R169.2, R170.2, R171.2, R172.2, R173.2, R174.2, R175.2, R176.2, R177.2
- new net: LED145.A, R145.2
- new net: D_141.2 (A), K_141.2
- new net: LED141.A, R141.2
- new net: LED148.A, R148.2
- new net: LED123.A, R123.2
- new net: LED138.A, R138.2
- new net: LED126.A, R126.2
- new net: D_106.2 (A), K_106.2
- new net: D_134.2 (A), K_134.2
- new net: D_137.2 (A), K_137.2
- new net: LED168.A, R168.2
- new net: D_156.2 (A), K_156.2
- new net: LED129.A, R129.2
- new net: D_154.2 (A), K_154.2
- new net: LED101.A, R101.2
- new net: LED176.A, R176.2
- new net: LED124.A, R124.2
- new net: D_148.2 (A), K_148.2
- new net: D_108.2 (A), K_108.2
- new net: D_103.2 (A), K_103.2
- new net: D_151.2 (A), K_151.2
- new net: D_119.2 (A), K_119.2
- new net: LED154.A, R154.2
- new net: D_152.2 (A), K_152.2
- new net: D_147.2 (A), K_147.2
- new net: LED151.A, R151.2
- new net: LED120.A, R120.2
- new net: D_129.2 (A), K_129.2
- new net: D_161.2 (A), K_161.2
- new net: D_116.2 (A), K_116.2
- new net: LED116.A, R116.2
- new net: D_170.2 (A), K_170.2
- new net: LED119.A, R119.2
- new net: D_107.2 (A), K_107.2
- new net: LED104.A, R104.2
- new net: LED172.A, R172.2
- new net: D_104.2 (A), K_104.2
- new net: LED166.A, R166.2
- new net: LED153.A, R153.2
- new net: LED161.A, R161.2
- new net: D_177.2 (A), K_177.2
- new net: LED114.A, R114.2
- new net: LED139.A, R139.2
- new net: LED115.A, R115.2
- new net: LED102.A, R102.2
- new net: D_162.2 (A), K_162.2
- new net: LED170.A, R170.2
- new net: D_146.2 (A), K_146.2
- new net: LED135.A, R135.2
- new net: D_115.2 (A), K_115.2
- new net: LED121.A, R121.2
- new net: LED132.A, R132.2
- new net: D_149.2 (A), K_149.2
- new net: LED156.A, R156.2
- new net: D_132.2 (A), K_132.2
- new net: LED164.A, R164.2
- new net: LED137.A, R137.2
- new net: LED158.A, R158.2
- new net: LED149.A, R149.2
- new net: LED103.A, R103.2
- new net: LED147.A, R147.2
- new net: LED169.A, R169.2
- new net: D_142.2 (A), K_142.2
- new net: LED130.A, R130.2
- new net: LED108.A, R108.2
- new net: LED113.A, R113.2
- new net: LED140.A, R140.2
- new net: LED143.A, R143.2
- new net: D_131.2 (A), K_131.2
- new net: LED146.A, R146.2
- new net: D_165.2 (A), K_165.2
- new net: D_175.2 (A), K_175.2
- new net: LED122.A, R122.2
- new net: D_111.2 (A), K_111.2
- new net: LED117.A, R117.2
- new net: D_139.2 (A), K_139.2
- new net: D_105.2 (A), K_105.2
- new net: D_159.2 (A), K_159.2
- new net: D_135.2 (A), K_135.2
- new net: D_112.2 (A), K_112.2
- new net: LED110.A, R110.2
- new net: LED127.A, R127.2
- new net: LED128.A, R128.2
- new net: LED173.A, R173.2
- new net: LED133.A, R133.2
- new net: D_126.2 (A), K_126.2
- new net: D_172.2 (A), K_172.2
- new net: D_168.2 (A), K_168.2
- new net: D_124.2 (A), K_124.2
- new net: D_169.2 (A), K_169.2
- new net: D_157.2 (A), K_157.2
- new net: Q1.1 (G), R5.1
- new net: D_122.2 (A), K_122.2
- new net: LED163.A, R163.2
- new net: D_173.2 (A), K_173.2
- new net: D_158.2 (A), K_158.2
- new net: LED167.A, R167.2
- new net: D_174.2 (A), K_174.2
- new net: D_150.2 (A), K_150.2
- new net: LED112.A, R112.2
- new net: LED105.A, R105.2
- new net: D_144.2 (A), K_144.2
- new net: LED155.A, R155.2
- new net: LED175.A, R175.2
- new net: D_109.2 (A), K_109.2
- new net: LED125.A, R125.2
- new net: D_110.2 (A), K_110.2
- new net: D_138.2 (A), K_138.2
- new net: LED144.A, R144.2
- new net: LED160.A, R160.2
- new net: D_102.2 (A), K_102.2
- new net: D_164.2 (A), K_164.2
- new net: LED165.A, R165.2
- new net: LED142.A, R142.2
- new net: D_163.2 (A), K_163.2
- new net: D_143.2 (A), K_143.2
- new net: LED118.A, R118.2
- new net: D_171.2 (A), K_171.2
- new net: D_127.2 (A), K_127.2
- new net: D_117.2 (A), K_117.2
- new net: LED150.A, R150.2
- new net: LED159.A, R159.2
- new net: D_121.2 (A), K_121.2
- new net: LED152.A, R152.2
- new net: LED136.A, R136.2
- new net: D_140.2 (A), K_140.2
- new net: LED111.A, R111.2
- new net: D_145.2 (A), K_145.2
- new net: D_118.2 (A), K_118.2
- new net: LED134.A, R134.2
- new net: D_166.2 (A), K_166.2
- new net: D_136.2 (A), K_136.2
- new net: LED131.A, R131.2
- new net: D_153.2 (A), K_153.2
- new net: D_113.2 (A), K_113.2
- new net: LED1.K, R7.1
- new net: LED174.A, R174.2
- new net: LED162.A, R162.2
- new net: LED171.A, R171.2
- new net: D_130.2 (A), K_130.2
- new net: D_125.2 (A), K_125.2
- new net: D_101.2 (A), K_101.2
- new net: D_176.2 (A), K_176.2
- new net: LED106.A, R106.2
- new net: LED107.A, R107.2
- new net: D_114.2 (A), K_114.2
- new net: D_167.2 (A), K_167.2
- new net: D_160.2 (A), K_160.2
- new net: D_120.2 (A), K_120.2
- new net: D_128.2 (A), K_128.2
- new net: LED177.A, R177.2
- new net: D_123.2 (A), K_123.2
- new net: LED157.A, R157.2
- new net: LED109.A, R109.2
- new net: D_133.2 (A), K_133.2
- new net: D_155.2 (A), K_155.2
Other:
- note added: "LEDs"
- moved on the sheet: FB401, J401, R401, R402, U3

Commit message: (WIP) rev2b work
Parts:
- removed R3: 10k, Resistor_SMD:R_0805_2012Metric, symbol Device:R_Small
- K_127: footprint acheron_MX_soldermask:MX200 -> acheron_MX_soldermask:MX200R
- U2: footprint acheron_Components:LQFP-48_7x7mm_P0.5mm -> acheron_Components:STM_UFQFPN-48_LQFP-48-1EP_7x7mm_P0.5mm_HandSoldering_ThermalReliefs
Connections:
- net COL0: no longer U2.10 (PA0-WKUP), U2.11 (PA1), U2.12 (PA2), U2.13 (PA3), U2.14 (PA4), U2.15 (PA5), U2.17 (PA7), U2.18 (PB0), U2.21 (B10), U2.25 (PB12), U2.27 (PB14), U2.3 (PC14_OSC32IN), U2.4 (PC15_OSC32OUT)
- net COL1: now also U2.3 (PC14_OSC32IN)
- net COL10: now also U2.18 (PB0)
- net COL11: now also U2.21 (B10)
- net COL12: now also U2.25 (PB12)
- net COL13: now also U2.27 (PB14)
- net COL2: now also U2.4 (PC15_OSC32OUT)
- net COL3: now also U2.10 (PA0-WKUP)
- net COL4: now also U2.11 (PA1)
- net COL5: now also U2.12 (PA2)
- net COL6: now also U2.13 (PA3)
- net COL7: now also U2.14 (PA4)
- net COL8: now also U2.15 (PA5)
- net COL9: now also U2.17 (PA7)
- net GNDPWR: now also J401.S (SHIELD); no longer J401.S1 (SHIELD)
- net VLED: now reaches Q1.3 (D), R101.1, R102.1, R103.1, R104.1, R105.1, R106.1, R107.1, R108.1, R109.1, R110.1, R111.1, R112.1, R113.1, R114.1, R115.1, R116.1, R117.1, R118.1, R119.1, R120.1, R121.1, R122.1, R123.1, R124.1, R125.1, R126.1, R127.1, R128.1, R129.1, R130.1, R131.1, R132.1, R133.1, R134.1, R135.1, R136.1, R137.1, R138.1, R139.1, R140.1, R141.1, R142.1, R143.1, R144.1, R145.1, R146.1, R147.1, R148.1, R149.1, R150.1, R151.1, R152.1, R153.1, R154.1, R155.1, R156.1, R157.1, R158.1, R159.1, R160.1, R161.1, R162.1, R163.1, R164.1, R165.1, R166.1, R167.1, R168.1, R169.1, R170.1, R171.1, R172.1, R173.1, R174.1, R175.1, R176.1, R177.1
Changed lines of the file:
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@@
     (stroke (width 0) (type solid) (color 0 0 0 0))
   )
-  (wire (pts (xy 139.7 69.85) (xy 142.24 69.85))
-    (stroke (width 0) (type default) (color 0 0 0 0))
-  )
   (wire (pts (xy 473.075 283.845) (xy 483.235 283.845))
     (stroke (width 0) (type default) (color 0 0 0 0))
@@
     (stroke (width 0.508) (type dash) (color 0 0 0 0))
   )
-  (wire (pts (xy 151.13 69.85) (xy 147.32 69.85))
-    (stroke (width 0) (type solid) (color 0 0 0 0))
-  )
   (wire (pts (xy 476.25 113.03) (xy 478.79 113.03))
     (stroke (width 0) (type default) (color 0 0 0 0))
@@
     (effects (font (size 1.27 1.27)) (justify left bottom))
   )
+  (label "VLED" (at 353.06 217.17 0)
+    (effects (font (size 2 2)) (justify left bottom))
+  )
   (global_label "SCL" (shape output) (at 248.285 39.37 90)
     (effects (font (size 1.27 1.27)) (justify left))
@@
     )
   )
-  (global_label "COL0" (shape input) (at 260.985 139.7 270) (fields_autoplaced)
+  (global_label "COL11" (shape input) (at 260.985 139.7 270) (fields_autoplaced)
     (effects (font (size 1.27 1.27)) (justify right))
-    (property "Intersheet References" "${INTERSHEET_REFS}" (id 0) (at 260.9056 147.1417 90)
+    (property "Intersheet References" "${INTERSHEET_REFS}" (id 0) (at 260.9056 148.3512 90)
       (effects (font (size 1.27 1.27)) (justify right) hide)
     )
@@
     )
   )
-  (global_label "COL0" (shape input) (at 201.295 130.81 180) (fields_autoplaced)
+  (global_label "COL5" (shape input) (at 201.295 130.81 180) (fields_autoplaced)
     (effects (font (size 1.27 1.27)) (justify right))
     (property "Intersheet References" "${INTERSHEET_REFS}" (id 0) (at 193.8533 130.7306 0)
@@
     )
   )
-  (global_label "COL0" (shape input) (at 222.885 139.7 270) (fields_autoplaced)
+  (global_label "COL8" (shape input) (at 222.885 139.7 270) (fields_autoplaced)
     (effects (font (size 1.27 1.27)) (justify right))
     (property "Intersheet References" "${INTERSHEET_REFS}" (id 0) (at 222.8056 147.1417 90)
@@
     )
   )
-  (global_label "COL0" (shape input) (at 288.925 119.38 0) (fields_autoplaced)
+  (global_label "COL13" (shape input) (at 288.925 119.38 0) (fields_autoplaced)
     (effects (font (size 1.27 1.27)) (justify left))
-    (property "Intersheet References" "${INTERSHEET_REFS}" (id 0) (at 296.3667 119.4594 0)
+    (property "Intersheet References" "${INTERSHEET_REFS}" (id 0) (at 297.5762 119.3006 0)
       (effects (font (size 1.27 1.27)) (justify left) hide)
     )
   )
-  (global_label "COL0" (shape input) (at 288.925 132.08 0) (fields_autoplaced)
+  (global_label "COL12" (shape input) (at 288.925 132.08 0) (fields_autoplaced)
     (effects (font (size 1.27 1.27)) (justify left))
-    (property "Intersheet References" "${INTERSHEET_REFS}" (id 0) (at 296.3667 132.1594 0)
+    (property "Intersheet References" "${INTERSHEET_REFS}" (id 0) (at 297.5762 132.0006 0)
       (effects (font (size 1.27 1.27)) (justify left) hide)
     )
@@
     )
   )
-  (global_label "COL0" (shape input) (at 201.295 124.46 180) (fields_autoplaced)
+  (global_label "COL4" (shape input) (at 201.295 124.46 180) (fields_autoplaced)
     (effects (font (size 1.27 1.27)) (justify right))
     (property "Intersheet References" "${INTERSHEET_REFS}" (id 0) (at 193.8533 124.3806 0)
@@
     )
   )
-  (global_label "COL0" (shape input) (at 201.295 118.11 180) (fields_autoplaced)
+  (global_label "COL3" (shape input) (at 201.295 118.11 180) (fields_autoplaced)
     (effects (font (size 1.27 1.27)) (justify right))
     (property "Intersheet References" "${INTERSHEET_REFS}" (id 0) (at 193.8533 118.0306 0)
@@
     )
   )
-  (global_label "COL0" (shape input) (at 235.585 139.7 270) (fields_autoplaced)
+  (global_label "COL9" (shape input) (at 235.585 139.7 270) (fields_autoplaced)
     (effects (font (size 1.27 1.27)) (justify right))
     (property "Intersheet References" "${INTERSHEET_REFS}" (id 0) (at 235.5056 147.1417 90)
@@
     )
   )
-  (global_label "COL0" (shape input) (at 201.295 73.66 180) (fields_autoplaced)
+  (global_label "COL1" (shape input) (at 201.295 73.66 180) (fields_autoplaced)
     (effects (font (size 1.27 1.27)) (justify right))
     (property "Intersheet References" "${INTERSHEET_REFS}" (id 0) (at 193.8533 73.5806 0)
@@
     )
   )
-  (global_label "COL0" (shape input) (at 241.935 139.7 270) (fields_autoplaced)
+  (global_label "COL10" (shape input) (at 241.935 139.7 270) (fields_autoplaced)
     (effects (font (size 1.27 1.27)) (justify right))
-    (property "Intersheet References" "${INTERSHEET_REFS}" (id 0) (at 241.8556 147.1417 90)
+    (property "Intersheet References" "${INTERSHEET_REFS}" (id 0) (at 241.8556 148.3512 90)
       (effects (font (size 1.27 1.27)) (justify right) hide)
     )
   )
-  (global_label "COL0" (shape input) (at 216.535 139.7 270) (fields_autoplaced)
+  (global_label "COL7" (shape input) (at 216.535 139.7 270) (fields_autoplaced)
     (effects (font (size 1.27 1.27)) (justify right))
     (property "Intersheet References" "${INTERSHEET_REFS}" (id 0) (at 216.4556 147.1417 90)
@@
     )
   )
-  (global_label "PB2{slash}BOOT1" (shape input) (at 139.7 69.85 180)
-    (effects (font (size 0.762 0.762)) (justify right))
-    (property "Intersheet References" "${INTERSHEET_REFS}" (id 0) (at 131.6639 69.9135 0)
-      (effects (font (size 0.762 0.762)) (justify right) hide)
-    )
-  )
   (global_label "SDA" (shape bidirectional) (at 68.58 52.705 0)
     (effects (font (size 0.762 0.762)) (justify left))
@@
     )
   )
-  (global_label "COL0" (shape input) (at 210.185 139.7 270) (fields_autoplaced)
+  (global_label "COL6" (shape input) (at 210.185 139.7 270) (fields_autoplaced)
     (effects (font (size 1.27 1.27)) (justify right))
     (property "Intersheet References" "${INTERSHEET_REFS}" (id 0) (at 210.1056 147.1417 90)
@@
     )
   )
-  (global_label "COL0" (shape input) (at 201.295 80.01 180) (fields_autoplaced)
+  (global_label "COL2" (shape input) (at 201.295 80.01 180) (fields_autoplaced)
     (effects (font (size 1.27 1.27)) (justify right))
     (property "Intersheet References" "${INTERSHEET_REFS}" (id 0) (at 193.8533 79.9306 0)
@@
       (effects (font (size 2.0066 2.0066) bold))
     )
-    (property "Footprint" "acheron_Components:LQFP-48_7x7mm_P0.5mm" (id 2) (at 243.205 111.125 0)
+    (property "Footprint" "acheron_Components:STM_UFQFPN-48_LQFP-48-1EP_7x7mm_P0.5mm_HandSoldering_ThermalReliefs" (id 2) (at 243.205 111.125 0)
       (effects (font (size 1.27 1.27)) hide)
     )
@@
     (pin "B7")
     (pin "B8")
-    (pin "S1")
+    (pin "S")
   )
   (symbol (lib_id "acheron_Symbols:Mechanical_Switch") (at 66.675 313.69 0) (unit 1)
@@
     (pin "1")
   )
-  (symbol (lib_id "Device:R_Small") (at 144.78 69.85 90) (unit 1)
-    (in_bom yes) (on_board yes)
-    (property "Reference" "R3" (id 0) (at 144.78 67.945 90)
-      (effects (font (size 0.7874 0.7874)))
-    )
-    (property "Value" "10k" (id 1) (at 144.78 69.85 90)
-      (effects (font (size 0.7874 0.7874)))
-    )
-    (property "Footprint" "Resistor_SMD:R_0805_2012Metric" (id 2) (at 144.78 69.85 0)
-      (effects (font (size 1.27 1.27)) hide)
-    )
-    (property "Datasheet" "~" (id 3) (at 144.78 69.85 0)
-      (effects (font (size 1.27 1.27)) hide)
-    )
-    (property "Package" "R0805" (id 4) (at 144.78 69.85 0)
-      (effects (font (size 1.27 1.27)) hide)
-    )
-    (pin "1")
-    (pin "2")
-  )
   (symbol (lib_id "acheron_Symbols:LED") (at 391.795 339.725 270) (unit 1)
     (in_bom no) (on_board yes) (fields_autoplaced)
@@
       (effects (font (size 0.762 0.762)) hide)
     )
-    (property "Footprint" "acheron_MX_soldermask:MX200" (id 2) (at 280.035 287.02 0)
+    (property "Footprint" "acheron_MX_soldermask:MX200R" (id 2) (at 280.035 287.02 0)
       (effects (font (size 1.27 1.27)) hide)
     )
@@
     (pin "K")
   )
-  (symbol (lib_id "power:GND") (at 151.13 69.85 90) (unit 1)
-    (in_bom yes) (on_board yes)
-    (property "Reference" "#PWR013" (id 0) (at 157.48 69.85 0)
-      (effects (font (size 1.27 1.27)) hide)
-    )
-    (property "Value" "GND" (id 1) (at 156.21 69.85 90)
-      (effects (font (size 0.762 0.762)))
-    )
-    (property "Footprint" "" (id 2) (at 151.13 69.85 0)
-      (effects (font (size 1.27 1.27)) hide)
-    )
-    (property "Datasheet" "" (id 3) (at 151.13 69.85 0)
-      (effects (font (size 1.27 1.27)) hide)
-    )
-    (pin "1")
-  )
   (symbol (lib_id "Device:D") (at 191.135 300.99 270) (unit 1)
     (in_bom yes) (on_board yes) (fields_autoplaced)
@@
       (reference "#PWR012") (unit 1) (value "GND") (footprint "")
     )
-    (path "/bb810b8e-693a-41b5-a46f-10831b7207b0"
-      (reference "#PWR013") (unit 1) (value "GND") (footprint "")
-    )
     (path "/d286e829-01bd-4856-945c-757ffc2b1518"
       (reference "#PWR014") (unit 1) (value "GND") (footprint "")
@@
     )
     (path "/a168f846-3d7f-4133-ae76-050d4853b222"
-      (reference "K_127") (unit 1) (value "Mechanical_Switch") (footprint "acheron_MX_soldermask:MX200")
+      (reference "K_127") (unit 1) (value "Mechanical_Switch") (footprint "acheron_MX_soldermask:MX200R")
     )
     (path "/df94f76c-603b-457e-9b56-41a30d439765"
@@
       (reference "R2") (unit 1) (value "4.7k") (footprint "Resistor_SMD:R_0402_1005Metric")
     )
-    (path "/49ac801b-5cc0-403c-a6c9-42bcc3b9a2f6"
-      (reference "R3") (unit 1) (value "10k") (footprint "Resistor_SMD:R_0805_2012Metric")
-    )
     (path "/733bdb7e-01f4-4787-850a-50e92efa88e6"
       (reference "R4") (unit 1) (value "1.5k") (footprint "Resistor_SMD:R_0402_1005Metric")
@@
     )
     (path "/02758f52-a200-46b5-b27b-07b7b8c9a0ad"
-      (reference "U2") (unit 1) (value "JOKER MCU") (footprint "acheron_Components:LQFP-48_7x7mm_P0.5mm")
+      (reference "U2") (unit 1) (value "JOKER MCU") (footprint "acheron_Components:STM_UFQFPN-48_LQFP-48-1EP_7x7mm_P0.5mm_HandSoldering_ThermalReliefs")
     )
     (path "/fc872784-61d7-4741-b47c-bf115445f57a"
