File: kicad/rev2b/BareDevRev2.kicad_pcb (KiCad board)
At the start: 2 copper layers, 80 x 60 mm, 19 parts, among them U1 BL24C256A-SFRC, U2 STM32F411CEU6, X1 ARM JTAG, Y1 7325-0800A2010-00

Commit message: initial rev2b schematic
Other:
- board text removed: "READ THE DOCUMENTATION."
- board text removed: "Whether you are using these files for a hobby project or plan to use it for actually selling PCBs, you MUST know what you are using and getting yourself into. Read the notes, the documentation and understand it fully. You may remove this message."
Changed lines of the file:
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@@
   (gr_line (start 623.749972 109.649999) (end 625.749972 107.649999) (layer "Cmts.User") (width 0.5))
   (gr_line (start 549.749972 164.649999) (end 559.749972 154.649999) (layer "Cmts.User") (width 0.5))
-  (gr_circle (center 235.749972 70.149999) (end 236.049972 70.149999) (layer "Cmts.User") (width 1) (fill none))
   (gr_line (start 467.749972 164.649999) (end 469.749972 162.649999) (layer "Cmts.User") (width 0.5))
   (gr_line (start 703.749972 9.649999) (end 713.749972 -0.350001) (layer "Cmts.User") (width 0.5))
@@
   (gr_line (start 527.749972 51.649999) (end 529.749972 49.649999) (layer "Cmts.User") (width 0.5))
   (gr_line (start 641.749972 101.649999) (end 643.749972 99.649999) (layer "Cmts.User") (width 0.5))
-  (gr_line (start 241.749972 72.149999) (end 235.749972 62.149999) (layer "Cmts.User") (width 1))
   (gr_line (start 633.749972 9.649999) (end 635.749972 7.649999) (layer "Cmts.User") (width 0.5))
   (gr_line (start 643.749972 109.649999) (end 645.749972 107.649999) (layer "Cmts.User") (width 0.5))
@@
   (gr_line (start 580.749972 104.649999) (end 585.749972 99.649999) (layer "Cmts.User") (width 0.5))
   (gr_line (start 683.749972 101.649999) (end 685.749972 99.649999) (layer "Cmts.User") (width 0.5))
-  (gr_line (start 235.749972 65.149999) (end 235.749972 68.149999) (layer "Cmts.User") (width 1))
   (gr_line (start 635.749972 9.649999) (end 637.749972 7.649999) (layer "Cmts.User") (width 0.5))
   (gr_line (start 517.749972 164.649999) (end 519.749972 162.649999) (layer "Cmts.User") (width 0.5))
@@
   (gr_line (start 565.749972 9.649999) (end 570.749972 4.649999) (layer "Cmts.User") (width 0.5))
   (gr_line (start 523.749972 156.649999) (end 525.749972 154.649999) (layer "Cmts.User") (width 0.5))
-  (gr_line (start 229.749972 72.149999) (end 241.749972 72.149999) (layer "Cmts.User") (width 1))
   (gr_line (start 585.749972 109.649999) (end 595.749972 99.649999) (layer "Cmts.User") (width 0.5))
   (gr_line (start 430.749972 4.649999) (end 435.749972 -0.350001) (layer "Cmts.User") (width 0.5))
@@
   (gr_line (start 433.749972 164.649999) (end 443.749972 154.649999) (layer "Cmts.User") (width 0.5))
   (gr_line (start 529.749972 156.649999) (end 531.749972 154.649999) (layer "Cmts.User") (width 0.5))
-  (gr_line (start 235.749972 62.149999) (end 229.749972 72.149999) (layer "Cmts.User") (width 1))
   (gr_line (start 455.749972 164.649999) (end 465.749972 154.649999) (layer "Cmts.User") (width 0.5))
   (gr_line (start 667.749972 1.649999) (end 669.749972 -0.350001) (layer "Cmts.User") (width 0.5))
@@
     (effects (font (size 1 1) (thickness 0.2)) (justify left))
   )
-  (gr_text "READ THE DOCUMENTATION." (at 215.249972 79.649999) (layer "Cmts.User")
-    (effects (font (size 2 2) (thickness 0.5)) (justify left))
-  )
   (gr_text "The actually used values can very well vary according to your specifications and the capabilities of the factory being used." (at 434.249972 119.649999) (layer "Cmts.User")
     (effects (font (size 1 1) (thickness 0.2)) (justify left))
@@
     (effects (font (size 1 1) (thickness 0.2)) (justify left))
   )
-  (gr_text "Whether you are using these files for a hobby project or plan to use it for actually selling PCBs, you MUST\nknow what you are using and getting yourself into. Read the notes, the documentation and understand it fully.\nYou may remove this message." (at 199.749972 84.649999) (layer "Cmts.User")
-    (effects (font (size 1 1) (thickness 0.2)) (justify left))
-  )
   (gr_text "(3) KiCAD allows custom user layers. Use those to indicate screw hole anchors/sizes, plate markings, stabilizer orientation. Document everything because" (at 590.749972 144.649999) (layer "Cmts.User")
     (effects (font (size 1 1) (thickness 0.2)) (justify left))
@@
     (effects (font (size 2 2) (thickness 0.5)) (justify left))
   )
-  (gr_text "IMPORTANT" (at 235.749972 75.149999) (layer "Cmts.User")
-    (effects (font (size 2 2) (thickness 0.5)))
-  )
   (gr_text "0.5" (at 676.749972 43.649999) (layer "Cmts.User")
